File: KiCad/EnvSensor-v2/EnvSensor-v2.sch (KiCad schematic (older format))
At the start: 155 parts, among them J1 Conn_01x06, J10 Conn_01x02, J2 Conn_01x02, J3 USB_B_Micro, J4 Conn_01x02, J5 Micro_SD_Card_Det, J6 Conn_01x02, J8 HPMA115C0-003, J9 Conn_01x02, P1 USB_C_Plug_USB2.0, Q1 IRLML2502, Q2 Si3407DV, Q3 AUiRLR3110Z, Q4 AO6804A, SW1 SW_Push, SW2 Reset, SW3 SW_Push, SW4 SW_Push, SW5 SW_Push, U1 STM32L451RETx, U10 LTC3440, U11 MCP1826S-5.0, U12 MCP1825S-3.3, U2 E-Ink_Waveshare_4.2, U3 SCD30, U4 SCD40, U5 BME280, U6 AP9101CK, U7 MCP73843-4.2, U8 BME280-Module, U9 LM2735XMF, Y1 16Hz, Y2 32768/12.5pF

Commit message: Work on pcb v2
Parts:
- added C44: 22u, Capacitor_SMD:C_1206_3216Metric, symbol Device:C
- added C45: 1u, Capacitor_SMD:C_0805_2012Metric, symbol Device:C
- added C?: 10u, Capacitor_SMD:C_0805_2012Metric, symbol Device:C
- J1: value Conn_01x06 -> JTAG; footprint Connector_PinHeader_2.54mm:PinHeader_1x06_P2.54mm_Horizontal -> Connector_PinHeader_2.54mm:PinHeader_1x06_P2.54mm_Vertical
- J8: footprint Connector_PinHeader_2.54mm:PinHeader_1x04_P2.54mm_Horizontal -> Connector_PinHeader_2.54mm:PinHeader_1x04_P2.54mm_Vertical
- JP4: footprint Jumper:SolderJumper-2_P1.3mm_Open_RoundedPad1.0x1.5mm -> Jumper:SolderJumper-2_P1.3mm_Bridged_RoundedPad1.0x1.5mm
- U1: value STM32L451RETx -> STM32L451RCT6
Connections:
- net +BATT: now also C?.1
- net BATTERY_MEASURE_ENABLE: now also U1.57 (PB5)
- net BATTERY_MEASURE_INPUT: now also U1.58 (PB6), C45.1
- net E_INK_BUSY: now also U1.27 (PB1)
- net E_INK_CD: now also U1.25 (PC5)
- net E_INK_RESET: now also U1.26 (PB0)
- net E_INK_SELECT: now also U1.24 (PC4)
- net GND: now also SW2.1, U12.2 (GND), C44.2, C45.2, C?.2; no longer SW2.2
- net HPMA_RX: now also U1.16 (PA2)
- net HPMA_TX: now also U1.17 (PA3)
- net LED_1: now also U1.11 (PC3)
- net LED_2: now also U1.10 (PC2)
- net LED_3: now also U1.9 (PC1)
- net LED_4: now also U1.8 (PC0)
- net MOSI: now also U1.23 (PA7)
- net NRST: now also SW2.2; no longer SW2.1
- net POWER_5V_ENABLE: now also U1.28 (PB2)
- net SCD30_READY: now also U1.44 (PA11)
- net SCK: now also U1.21 (PA5)
- net SCL: now also U1.42 (PA9)
- net SDA: now also U1.43 (PA10)
- net SDIO_CLK: now also U1.53 (PC12)
- net SDIO_CMD: now also U1.54 (PD2)
- net SDIO_DATA0: now also U1.39 (PC8)
- net SDIO_DATA1: now also U1.40 (PC9)
- net SDIO_DATA2: now also U1.51 (PC10)
- net SDIO_DATA3: now also U1.52 (PC11)
- net SDIO_DETECT: now also U1.38 (PC7)
- net SDIO_POWER_ENABLE: now also U1.37 (PC6)
- net SWITCH_1: now also U1.33 (PB12)
- net SWITCH_2: now also U1.34 (PB13)
- net SWITCH_3: now also U1.35 (PB14)
- net SWITCH_4: now also U1.36 (PB15)
- net at C37.1, C38.1, C39.1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: now also U12.1 (VI); no longer J9.1 (Pin_1), JP6.1
- net at U12.3 (VO): now also J9.1 (Pin_1), JP6.1, C44.1
Other:
- moved on the sheet: C29, C30, C33, C37, C38, C39, C40, C43, D14, D16, J9, JP4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

Commit message: Finishing touches
Parts:
- added J7: I2C, Connector_PinSocket_2.54mm:PinSocket_1x04_P2.54mm_Vertical, symbol Connector_Generic:Conn_01x04
- gave numbers to parts that had none: 1
Connections:
- net +3V3: now also J7.4 (Pin_4)
- net GND: now also J7.3 (Pin_3)
- net SCD30_READY: now also U1.41 (PA8); no longer U1.44 (PA11)
- net SCL: now also J7.2 (Pin_2)
- net SDA: now also J7.1 (Pin_1)
Other:
- note added: "I2C"
- moved on the sheet: J1, R12, R13
Changed lines of the file:
@@
 L Connector_Generic:Conn_01x06 J1
 U 1 1 615007AE
-P 4100 7900
-F 0 "J1" H 4180 7892 50  0000 L CNN
-F 1 "JTAG" H 4180 7801 50  0000 L CNN
-F 2 "Connector_PinHeader_2.54mm:PinHeader_1x06_P2.54mm_Vertical" H 4100 7900 50  0001 C CNN
-F 3 "~" H 4100 7900 50  0001 C CNN
-	1    4100 7900
+P 2800 8100
+F 0 "J1" H 2880 8092 50  0000 L CNN
+F 1 "JTAG" H 2880 8001 50  0000 L CNN
+F 2 "Connector_PinHeader_2.54mm:PinHeader_1x06_P2.54mm_Vertical" H 2800 8100 50  0001 C CNN
+F 3 "~" H 2800 8100 50  0001 C CNN
+	1    2800 8100
 	1    0    0    -1
 $EndComp
@@
 L power:+3.3V #PWR0117
 U 1 1 6150213F
-P 3700 7700
-F 0 "#PWR0117" H 3700 7550 50  0001 C CNN
-F 1 "+3.3V" V 3715 7828 50  0000 L CNN
-F 2 "" H 3700 7700 50  0001 C CNN
-F 3 "" H 3700 7700 50  0001 C CNN
-	1    3700 7700
+P 2400 7900
+F 0 "#PWR0117" H 2400 7750 50  0001 C CNN
+F 1 "+3.3V" V 2415 8028 50  0000 L CNN
+F 2 "" H 2400 7900 50  0001 C CNN
+F 3 "" H 2400 7900 50  0001 C CNN
+	1    2400 7900
 	0    -1   -1   0
 $EndComp
-Text GLabel 3700 7800 0    44   Input ~ 0
+Text GLabel 2400 8000 0    44   Input ~ 0
 SWCLK
-Text GLabel 3700 8000 0    44   Input ~ 0
+Text GLabel 2400 8200 0    44   Input ~ 0
 SWDIO
-Text GLabel 3700 8100 0    44   Input ~ 0
+Text GLabel 2400 8300 0    44   Input ~ 0
 NRST
-Text GLabel 3700 8200 0    44   Input ~ 0
+Text GLabel 2400 8400 0    44   Input ~ 0
 SWO
 Wire Wire Line
-	3700 8200 3900 8200
+	2400 8400 2600 8400
 Wire Wire Line
-	3700 8100 3900 8100
+	2400 8300 2600 8300
 Wire Wire Line
-	3700 8000 3900 8000
+	2400 8200 2600 8200
 Wire Wire Line
-	3700 7800 3900 7800
+	2400 8000 2600 8000
 Wire Wire Line
-	3700 7700 3900 7700
+	2400 7900 2600 7900
 $Comp
 L power:GND #PWR0118
 U 1 1 6151689F
-P 3700 7900
-F 0 "#PWR0118" H 3700 7650 50  0001 C CNN
-F 1 "GND" V 3705 7772 50  0000 R CNN
-F 2 "" H 3700 7900 50  0001 C CNN
-F 3 "" H 3700 7900 50  0001 C CNN
-	1    3700 7900
+P 2400 8100
+F 0 "#PWR0118" H 2400 7850 50  0001 C CNN
+F 1 "GND" V 2405 7972 50  0000 R CNN
+F 2 "" H 2400 8100 50  0001 C CNN
+F 3 "" H 2400 8100 50  0001 C CNN
+	1    2400 8100
 	0    1    1    0
 $EndComp
 Wire Wire Line
-	3700 7900 3900 7900
-Text Notes 3150 7350 0    118  ~ 0
+	2400 8100 2600 8100
+Text Notes 1850 7550 0    118  ~ 0
 JTAG Connector
 Text GLabel 4900 4300 2    44   Input ~ 0
@@
 Text GLabel 4900 3900 2    44   Input ~ 0
 SDA
-Text GLabel 4900 4000 2    44   Input ~ 0
+Text GLabel 4900 3700 2    44   Input ~ 0
 SCD30_READY
 Text Notes -5750 5200 2    118  ~ 0
@@
 L Device:R R12
 U 1 1 650B0665
-P 5150 1300
-F 0 "R12" H 5350 1250 50  0000 R CNN
-F 1 "10k" H 5350 1350 50  0000 R CNN
-F 2 "Resistor_SMD:R_0805_2012Metric" V 5080 1300 50  0001 C CNN
-F 3 "~" H 5150 1300 50  0001 C CNN
-	1    5150 1300
+P 5300 8200
+F 0 "R12" H 5500 8150 50  0000 R CNN
+F 1 "10k" H 5500 8250 50  0000 R CNN
+F 2 "Resistor_SMD:R_0805_2012Metric" V 5230 8200 50  0001 C CNN
+F 3 "~" H 5300 8200 50  0001 C CNN
+	1    5300 8200
 	-1   0    0    1
 $EndComp
-Text GLabel 5150 1450 3    44   Input ~ 0
+Text GLabel 5100 8550 0    44   Input ~ 0
 SCL
-Text GLabel 5250 1450 3    44   Input ~ 0
+Text GLabel 5100 8450 0    44   Input ~ 0
 SDA
 $Comp
 L power:+3.3V #PWR0174
 U 1 1 651554A7
-P 5200 1050
-F 0 "#PWR0174" H 5200 900 50  0001 C CNN
-F 1 "+3.3V" H 5215 1223 50  0000 C CNN
-F 2 "" H 5200 1050 50  0001 C CNN
-F 3 "" H 5200 1050 50  0001 C CNN
-	1    5200 1050
+P 5350 7950
+F 0 "#PWR0174" H 5350 7800 50  0001 C CNN
+F 1 "+3.3V" H 5365 8123 50  0000 C CNN
+F 2 "" H 5350 7950 50  0001 C CNN
+F 3 "" H 5350 7950 50  0001 C CNN
+	1    5350 7950
 	1    0    0    -1
 $EndComp
@@
 L Device:R R13
 U 1 1 65155977
-P 5250 1300
-F 0 "R13" H 5180 1254 50  0000 R CNN
-F 1 "10k" H 5180 1345 50  0000 R CNN
-F 2 "Resistor_SMD:R_0805_2012Metric" V 5180 1300 50  0001 C CNN
-F 3 "~" H 5250 1300 50  0001 C CNN
-	1    5250 1300
+P 5400 8200
+F 0 "R13" H 5330 8154 50  0000 R CNN
+F 1 "10k" H 5330 8245 50  0000 R CNN
+F 2 "Resistor_SMD:R_0805_2012Metric" V 5330 8200 50  0001 C CNN
+F 3 "~" H 5400 8200 50  0001 C CNN
+	1    5400 8200
 	-1   0    0    1
 $EndComp
 Wire Wire Line
-	5150 1150 5150 1100
+	5300 8050 5300 8000
 Wire Wire Line
-	5150 1100 5200 1100
+	5300 8000 5350 8000
 Wire Wire Line
-	5250 1100 5250 1150
+	5400 8000 5400 8050
 Wire Wire Line
-	5200 1100 5200 1050
-Connection ~ 5200 1100
+	5350 8000 5350 7950
+Connection ~ 5350 8000
 Wire Wire Line
-	5200 1100 5250 1100
+	5350 8000 5400 8000
 Text Notes -5750 5550 2    118  ~ 0
 SCD40
@@
 	3100 5300 3300 5300
 Wire Wire Line
-	4900 4000 4600 4000
-Wire Wire Line
 	4900 5800 4600 5800
 Wire Wire Line
@@
 	4900 4800 4600 4800
 $Comp
-L Device:C C?
+L Device:C C46
 U 1 1 63B41E8E
 P 18400 2150
-F 0 "C?" H 18450 2250 50  0000 L CNN
+F 0 "C46" H 18450 2250 50  0000 L CNN
 F 1 "10u" H 18450 2050 50  0000 L CNN
 F 2 "Capacitor_SMD:C_0805_2012Metric" H 18438 2000 50  0001 C CNN
@@
 Wire Wire Line
 	18400 2400 18650 2400
+Wire Wire Line
+	4600 3700 4900 3700
+$Comp
+L Connector_Generic:Conn_01x04 J7
+U 1 1 64774EC8
+P 5750 8550
+F 0 "J7" H 5830 8542 50  0000 L CNN
+F 1 "I2C" H 5830 8451 50  0000 L CNN
+F 2 "Connector_PinSocket_2.54mm:PinSocket_1x04_P2.54mm_Vertical" H 5750 8550 50  0001 C CNN
+F 3 "~" H 5750 8550 50  0001 C CNN
+	1    5750 8550
+	1    0    0    -1
+$EndComp
+Wire Wire Line
+	5100 8450 5400 8450
+Wire Wire Line
+	5100 8550 5300 8550
+Wire Wire Line
+	5400 8350 5400 8450
+Connection ~ 5400 8450
+Wire Wire Line
+	5400 8450 5550 8450
+Wire Wire Line
+	5300 8350 5300 8550
+Connection ~ 5300 8550
+Wire Wire Line
+	5300 8550 5550 8550
+$Comp
+L power:+3.3V #PWR0178
+U 1 1 649F2DDE
+P 5400 8750
+F 0 "#PWR0178" H 5400 8600 50  0001 C CNN
+F 1 "+3.3V" H 5415 8923 50  0000 C CNN
+F 2 "" H 5400 8750 50  0001 C CNN
+F 3 "" H 5400 8750 50  0001 C CNN
+	1    5400 8750
+	0    -1   -1   0
+$EndComp
+$Comp
+L power:GND #PWR0179
+U 1 1 649F3616
+P 5400 8650
+F 0 "#PWR0179" H 5400 8400 50  0001 C CNN
+F 1 "GND" H 5405 8477 50  0000 C CNN
+F 2 "" H 5400 8650 50  0001 C CNN
+F 3 "" H 5400 8650 50  0001 C CNN
+	1    5400 8650
+	0    1    1    0
+$EndComp
+Wire Wire Line
+	5400 8650 5550 8650
+Wire Wire Line
+	5400 8750 5550 8750
+Text Notes 5250 7550 0    118  ~ 0
+I2C
 $EndSCHEMATC

Commit message: pcb finishing touches
Parts:
- added R40: 30k, Resistor_SMD:R_0805_2012Metric, symbol Device:R
- D14: footprint Diode_SMD:D_SOD-323 -> Diode_SMD:D_SOD-323_HandSoldering
- J5: footprint Connector_Card:microSD_HC_Hirose_DM3BT-DSF-PEJS -> Connector_Card:microSD_HC_Hirose_DM3AT-SF-PEJM5
- R28: footprint Resistor_SMD:R_0805_2012Metric -> Resistor_SMD:R_0603_1608Metric
- R32: value 60k4 -> 30k
- R37: value 73k2 -> 47k
Connections:
- net GND: now also R40.2; no longer R32.2
- net SDIO_DETECT: now also U1.61 (PB8); no longer U1.38 (PC7)
- net SDIO_POWER_ENABLE: now also U1.62 (PB9); no longer U1.37 (PC6)
- net VBAT: now reaches C11.1, U1.1 (VBAT)
- net SD_3V3: now reaches C18.2, C19.2, J5.6 (VSS), Q2.4 (S), R19.2, R20.2, R21.2, R23.2, R24.2
- new net: R32.2, R40.1
- no-connect marks 11 -> 25
Other:
- note added: "Imax=110mA | 250mA\nPmax=0.4V*110mA | 0.4V*250mA\nPmax=44mW | 100mW"
- note added: "Imax=80mA\nPmax=0.5V*80mA=40mW"
- note added: "Pmax=(5.0V-2.5V)*0.5A=1.25W\nRja=50C/W"
- note added: "Vout=1.22*(1+R1/R2)\nR1=300k, R2=173.2k, Vo=3.33\nR1=300k, R2=147k, Vo=3.71"
- note removed: "Pmax=(5.0V-2.5V)*0.5A=1.25W\n"
- note removed: "Replace with DMG6968UDM-7"
Changed lines of the file:
@@
 1. Each part should allow to measure its power consumption\n2.\n\nEnhancements from v1.\n1. Reset button\n2. Button to start battery protection after power loss\n3. Solution to measure voltage at battery
 $Comp
-L MCU_ST_STM32L4:STM32L451RETx U1
-U 1 1 613A4072
-P 4000 4500
-F 0 "U1" H 4350 2750 50  0000 C CNN
-F 1 "STM32L451RCT6" H 4450 2650 50  0000 C CNN
-F 2 "Package_QFP:LQFP-64_10x10mm_P0.5mm" H 3400 2800 50  0001 R CNN
-F 3 "http://www.st.com/st-web-ui/static/active/en/resource/technical/document/datasheet/DM00340475.pdf" H 4000 4500 50  0001 C CNN
-	1    4000 4500
-	1    0    0    -1
-$EndComp
-$Comp
 L Transistor_FET:IRLML2060 Q1
 U 1 1 61413219
@@
 Text Notes 7850 11300 0    118  ~ 0
 E-Ink Display
-Text Notes 16850 2250 0    44   ~ 0
-Replace with DMG6968UDM-7
 $Comp
 L Device:R R29
@@
 F 0 "R28" V 14493 5250 50  0000 C CNN
 F 1 "100k" V 14584 5250 50  0000 C CNN
-F 2 "Resistor_SMD:R_0805_2012Metric" V 14630 5250 50  0001 C CNN
+F 2 "Resistor_SMD:R_0603_1608Metric" V 14630 5250 50  0001 C CNN
 F 3 "~" H 14700 5250 50  0001 C CNN
 	1    14700 5250
@@
 Connection ~ 16250 4050
 Text Notes 15850 3800 0    44   ~ 0
-Pmax=(5.0V-2.5V)*0.5A=1.25W\n
+Pmax=(5.0V-2.5V)*0.5A=1.25W\nRja=50C/W
 Wire Wire Line
 	14150 4200 14150 4050
@@
 F 0 "J5" H 12550 15067 50  0000 C CNN
 F 1 "Micro_SD_Card_Det" H 12550 14976 50  0000 C CNN
-F 2 "Connector_Card:microSD_HC_Hirose_DM3BT-DSF-PEJS" H 14650 14950 50  0001 C CNN
+F 2 "Connector_Card:microSD_HC_Hirose_DM3AT-SF-PEJM5" H 14650 14950 50  0001 C CNN
 F 3 "https://www.hirose.com/product/en/download_file/key_name/DM3/category/Catalog/doc_file_id/49662/?file_category_id=4&item_id=195&is_series=1" H 12600 14350 50  0001 C CNN
 	1    12600 14250
@@
 Text GLabel 3100 5800 0    44   Input ~ 0
 SDIO_CLK
-Text GLabel 3100 5200 0    44   Input ~ 0
+Text GLabel 4900 5500 2    44   Input ~ 0
 SDIO_POWER_ENABLE
-Text GLabel 3100 5300 0    44   Input ~ 0
+Text GLabel 4900 5400 2    44   Input ~ 0
 SDIO_DETECT
 $Comp
@@
 F 0 "D14" H 19150 1434 50  0000 C CNN
 F 1 "PMEG2010AEJ" H 19200 1550 50  0000 C CNN
-F 2 "Diode_SMD:D_SOD-323" H 19150 1650 50  0001 C CNN
+F 2 "Diode_SMD:D_SOD-323_HandSoldering" H 19150 1650 50  0001 C CNN
 F 3 "~" H 19150 1650 50  0001 C CNN
 	1    19150 1650
@@
 L power:GND #PWR0156
 U 1 1 62B2F64D
-P 19350 2650
-F 0 "#PWR0156" H 19350 2400 50  0001 C CNN
-F 1 "GND" H 19355 2477 50  0000 C CNN
-F 2 "" H 19350 2650 50  0001 C CNN
-F 3 "" H 19350 2650 50  0001 C CNN
-	1    19350 2650
+P 19350 2950
+F 0 "#PWR0156" H 19350 2700 50  0001 C CNN
+F 1 "GND" H 19355 2777 50  0000 C CNN
+F 2 "" H 19350 2950 50  0001 C CNN
+F 3 "" H 19350 2950 50  0001 C CNN
+	1    19350 2950
 	1    0    0    -1
 $EndComp
@@
 P 21150 2400
 F 0 "R37" H 20900 2450 50  0000 L CNN
-F 1 "73k2" H 20850 2350 50  0000 L CNN
+F 1 "47k" H 20850 2350 50  0000 L CNN
 F 2 "Resistor_SMD:R_0805_2012Metric" V 21080 2400 50  0001 C CNN
 F 3 "~" H 21150 2400 50  0001 C CNN
@@
 P 19350 2500
 F 0 "R32" H 19420 2546 50  0000 L CNN
-F 1 "60k4" H 19420 2455 50  0000 L CNN
+F 1 "30k" H 19420 2455 50  0000 L CNN
 F 2 "Resistor_SMD:R_0805_2012Metric" V 19280 2500 50  0001 C CNN
 F 3 "~" H 19350 2500 50  0001 C CNN
@@
 	4600 3900 4900 3900
 Wire Wire Line
-	3100 5200 3300 5200
-Wire Wire Line
-	3100 5300 3300 5300
-Wire Wire Line
 	4900 5800 4600 5800
 Wire Wire Line
@@
 Text Notes 5250 7550 0    118  ~ 0
 I2C
+Text Notes 21350 3750 0    44   ~ 0
+Imax=80mA\nPmax=0.5V*80mA=40mW
+Text Notes 19750 3050 0    44   ~ 0
+Vout=1.22*(1+R1/R2)\nR1=300k, R2=173.2k, Vo=3.33\nR1=300k, R2=147k, Vo=3.71
+Text Notes 21300 1350 0    44   ~ 0
+Imax=110mA | 250mA\nPmax=0.4V*110mA | 0.4V*250mA\nPmax=44mW | 100mW
+$Comp
+L Device:R R40
+U 1 1 6197DC55
+P 19350 2800
+F 0 "R40" H 19420 2846 50  0000 L CNN
+F 1 "30k" H 19420 2755 50  0000 L CNN
+F 2 "Resistor_SMD:R_0805_2012Metric" V 19280 2800 50  0001 C CNN
+F 3 "~" H 19350 2800 50  0001 C CNN
+	1    19350 2800
+	1    0    0    -1
+$EndComp
+Text Label 11650 12850 2    44   ~ 0
+SD_3V3
+Text Label 3700 2200 0    44   ~ 0
+VBAT
+Wire Wire Line
+	4900 5400 4600 5400
+Wire Wire Line
+	4600 5500 4900 5500
+$Comp
+L MCU_ST_STM32L4:STM32L451RETx U1
+U 1 1 613A4072
+P 4000 4500
+F 0 "U1" H 4350 2750 50  0000 C CNN
+F 1 "STM32L451RCT6" H 4450 2650 50  0000 C CNN
+F 2 "Package_QFP:LQFP-64_10x10mm_P0.5mm" H 3400 2800 50  0001 R CNN
+F 3 "http://www.st.com/st-web-ui/static/active/en/resource/technical/document/datasheet/DM00340475.pdf" H 4000 4500 50  0001 C CNN
+	1    4000 4500
+	1    0    0    -1
+$EndComp
+NoConn ~ 3300 5200
+NoConn ~ 3300 5300
+NoConn ~ 3300 5900
+NoConn ~ 4600 5700
+NoConn ~ 4600 5600
+NoConn ~ 4600 5300
+NoConn ~ 4600 5000
+NoConn ~ 4600 4400
+NoConn ~ 4600 4100
+NoConn ~ 4600 4000
+NoConn ~ 4600 3500
+NoConn ~ 4600 3300
+NoConn ~ 4600 3000
+NoConn ~ 4600 2900
 $EndSCHEMATC

Commit message: Finishing
Parts:
- added SW6: Start, Button_Switch_SMD:SW_SPST_CK_RS282G05A3, symbol Switch:SW_Push
- added U13: ESP-12S, JPComms:ESP-12S, symbol myLib:ESP-12S
Connections:
- net +3V3: now also U13.8 (VCC)
- net -BATT: now also SW6.1
- net GND: now also SW6.2, U13.9 (GND)
- net WIFI_RX: now reaches U1.29 (PB10)
- net WIFI_RX: now also U13.15 (RXD0)
- net WFI_TX: now reaches U1.30 (PB11)
- net WFI_TX: now also U13.16 (TXD0)
- net WIFI_RESET: now reaches U1.44 (PA11)
- net WIFI_RESET: now also U13.1 (Reset)
- net WIFI_ENABLE: now reaches U1.45 (PA12)
- net WIFI_ENABLE: now also U13.3 (EN)
- no-connect marks 25 -> 31
Other:
- note added: "WiFi"
Changed lines of the file:
@@
 L power:+BATT #PWR0103
 U 1 1 61447599
-P 16650 1500
-F 0 "#PWR0103" H 16650 1350 50  0001 C CNN
-F 1 "+BATT" V 16665 1628 50  0000 L CNN
-F 2 "" H 16650 1500 50  0001 C CNN
-F 3 "" H 16650 1500 50  0001 C CNN
-	1    16650 1500
+P 17000 1500
+F 0 "#PWR0103" H 17000 1350 50  0001 C CNN
+F 1 "+BATT" V 17015 1628 50  0000 L CNN
+F 2 "" H 17000 1500 50  0001 C CNN
+F 3 "" H 17000 1500 50  0001 C CNN
+	1    17000 1500
 	0    1    1    0
 $EndComp
@@
 L power:-BATT #PWR0104
 U 1 1 61448150
-P 16650 2850
-F 0 "#PWR0104" H 16650 2700 50  0001 C CNN
-F 1 "-BATT" V 16665 2978 50  0000 L CNN
-F 2 "" H 16650 2850 50  0001 C CNN
-F 3 "" H 16650 2850 50  0001 C CNN
-	1    16650 2850
+P 17000 2850
+F 0 "#PWR0104" H 17000 2700 50  0001 C CNN
+F 1 "-BATT" V 17015 2978 50  0000 L CNN
+F 2 "" H 17000 2850 50  0001 C CNN
+F 3 "" H 17000 2850 50  0001 C CNN
+	1    17000 2850
 	0    1    1    0
 $EndComp
@@
 Connection ~ 14150 1950
 Wire Wire Line
-	16650 1500 14150 1500
+	17000 1500 14150 1500
 Wire Wire Line
 	14150 1500 14150 1600
 Wire Wire Line
-	16650 2850 16150 2850
+	17000 2850 16800 2850
 Wire Wire Line
 	14150 2850 14150 2350
@@
 L power:GND #PWR0105
 U 1 1 61452FF2
-P 16700 1800
-F 0 "#PWR0105" H 16700 1550 50  0001 C CNN
-F 1 "GND" V 16705 1672 50  0000 R CNN
-F 2 "" H 16700 1800 50  0001 C CNN
-F 3 "" H 16700 1800 50  0001 C CNN
-	1    16700 1800
+P 17000 1800
+F 0 "#PWR0105" H 17000 1550 50  0001 C CNN
+F 1 "GND" V 17005 1672 50  0000 R CNN
+F 2 "" H 17000 1800 50  0001 C CNN
+F 3 "" H 17000 1800 50  0001 C CNN
+	1    17000 1800
 	0    -1   -1   0
 $EndComp
 Wire Wire Line
-	16700 1800 16150 1800
+	17000 1800 16800 1800
 Wire Wire Line
 	14450 1800 14450 2300
@@
 Wire Wire Line
 	16150 1800 14450 1800
-Text Notes 17150 2900 0    50   ~ 0
+Text Notes 17250 1450 0    50   ~ 0
 AP9101CK-AHTRG1\nVcu=4.425V\nVdl=2.5V\nVdoc=75mV\nVcoc=-75mV
 Text Notes 14050 1050 0    118  ~ 0
@@
 	9850 10900 9850 13250
 Wire Notes Line
-	9850 13250 7250 13250
-Wire Notes Line
 	7250 13250 7250 10900
 Wire Notes Line
@@
 NoConn ~ 3300 5300
 NoConn ~ 3300 5900
-NoConn ~ 4600 5700
-NoConn ~ 4600 5600
 NoConn ~ 4600 5300
 NoConn ~ 4600 5000
 NoConn ~ 4600 4400
-NoConn ~ 4600 4100
-NoConn ~ 4600 4000
 NoConn ~ 4600 3500
 NoConn ~ 4600 3300
 NoConn ~ 4600 3000
 NoConn ~ 4600 2900
+$Comp
+L Switch:SW_Push SW6
+U 1 1 624FC7DB
+P 16800 2300
+F 0 "SW6" V 16900 2600 50  0000 R CNN
+F 1 "Start" V 16700 2650 50  0000 R CNN
+F 2 "Button_Switch_SMD:SW_SPST_CK_RS282G05A3" H 16800 2500 50  0001 C CNN
+F 3 "~" H 16800 2500 50  0001 C CNN
+	1    16800 2300
+	0    1    -1   0
+$EndComp
+Wire Wire Line
+	16800 2100 16800 1800
+Connection ~ 16800 1800
+Wire Wire Line
+	16800 1800 16150 1800
+Wire Wire Line
+	16800 2500 16800 2850
+Connection ~ 16800 2850
+Wire Wire Line
+	16800 2850 16150 2850
+$Comp
+L myLib:ESP-12S U13
+U 1 1 629C2441
+P 15150 12250
+F 0 "U13" H 15150 12958 40  0000 C CNN
+F 1 "ESP-12S" H 15150 12882 40  0000 C CNN
+F 2 "JPComms:ESP-12S" H 15000 12150 60  0001 C CNN
+F 3 "" H 15000 12150 60  0000 C CNN
+	1    15150 12250
+	1    0    0    -1
+$EndComp
+$Comp
+L power:+3.3V #PWR0180
+U 1 1 629C3105
+P 15150 11700
+F 0 "#PWR0180" H 15150 11550 50  0001 C CNN
+F 1 "+3.3V" H 15165 11873 50  0000 C CNN
+F 2 "" H 15150 11700 50  0001 C CNN
+F 3 "" H 15150 11700 50  0001 C CNN
+	1    15150 11700
+	1    0    0    -1
+$EndComp
+$Comp
+L power:GND #PWR0181
+U 1 1 629C3350
+P 15150 12800
+F 0 "#PWR0181" H 15150 12550 50  0001 C CNN
+F 1 "GND" H 15155 12627 50  0000 C CNN
+F 2 "" H 15150 12800 50  0001 C CNN
+F 3 "" H 15150 12800 50  0001 C CNN
+	1    15150 12800
+	1    0    0    -1
+$EndComp
+NoConn ~ 15550 11850
+NoConn ~ 15550 11950
+NoConn ~ 15550 12050
+NoConn ~ 15550 12150
+NoConn ~ 15550 12250
+NoConn ~ 15550 12350
+NoConn ~ 15550 12450
+NoConn ~ 15550 12550
+NoConn ~ 15550 12650
+NoConn ~ 14750 12600
+Text GLabel 14600 11900 0    44   Input ~ 0
+WIFI_RESET
+Text GLabel 14600 12050 0    44   Input ~ 0
+WIFI_ENABLE
+Text GLabel 14600 12250 0    44   Input ~ 0
+WIFI_RX
+Text GLabel 14600 12350 0    44   Input ~ 0
+WFI_TX
+Wire Wire Line
+	14600 11900 14750 11900
+Wire Wire Line
+	14600 12050 14750 12050
+Wire Wire Line
+	14600 12250 14750 12250
+Wire Wire Line
+	14600 12350 14750 12350
+Wire Notes Line
+	9850 13250 7250 13250
+Wire Notes Line
+	16200 10900 16200 13250
+Wire Notes Line
+	16200 13250 13850 13250
+Wire Notes Line
+	13850 13250 13850 10900
+Wire Notes Line
+	13850 10900 16200 10900
+Text Notes 14850 11300 0    118  ~ 0
+WiFi
+Text GLabel 4900 4000 2    44   Input ~ 0
+WIFI_RESET
+Text GLabel 4900 4100 2    44   Input ~ 0
+WIFI_ENABLE
+Text GLabel 4900 5600 2    44   Input ~ 0
+WIFI_RX
+Text GLabel 4900 5700 2    44   Input ~ 0
+WFI_TX
+Wire Wire Line
+	4900 5700 4600 5700
+Wire Wire Line
+	4600 5600 4900 5600
+Wire Wire Line
+	4600 4000 4900 4000
+Wire Wire Line
+	4600 4100 4900 4100
 $EndSCHEMATC

Commit message: STM32CubeIDE/EnvSensorV2 introduced
Parts:
- Q3: value AUiRLR3110Z -> IRFR9024
Other:
- note added: "Bugs"
- note added: "NO analog input at PB6/58\nAvailable inputs: 14,15,20,22"
- note added: "Pmax=(5.0V-2.5V)*0.5A=1.25W\nRja=50C/W\ndeltaT=62.5C"
- note added: "Vmax=4.3V\n"
- note removed: "Pmax=(5.0V-2.5V)*0.5A=1.25W\nRja=50C/W"
Changed lines of the file:
@@
 Connection ~ 16250 4050
 Text Notes 15850 3800 0    44   ~ 0
-Pmax=(5.0V-2.5V)*0.5A=1.25W\nRja=50C/W
+Pmax=(5.0V-2.5V)*0.5A=1.25W\nRja=50C/W\ndeltaT=62.5C
 Wire Wire Line
 	14150 4200 14150 4050
@@
 P 15550 4150
 F 0 "Q3" V 15892 4150 50  0000 C CNN
-F 1 "AUiRLR3110Z" V 15801 4150 50  0000 C CNN
+F 1 "IRFR9024" V 15801 4150 50  0000 C CNN
 F 2 "Package_TO_SOT_SMD:TO-252-2" H 15750 4250 50  0001 C CNN
 F 3 "~" H 15550 4150 50  0001 C CNN
@@
 Wire Wire Line
 	4600 4100 4900 4100
+Text Notes 11350 2000 0    44   ~ 0
+Vmax=4.3V\n
+Text Notes -3700 1900 0    44   ~ 0
+NO analog input at PB6/58\nAvailable inputs: 14,15,20,22
+Text Notes -3700 1600 0    118  ~ 0
+Bugs
 $EndSCHEMATC

Commit message: bme280
Parts:
- U5: value BME280 -> BMP280
Connections:
- net BMP280_VCC: now reaches C20.1, C21.1, J6.1 (Pin_1), JP3.1, U5.2 (CSB), U5.6 (VDDIO), U5.8 (VDD), U8.1 (VDD), U8.5 (CSB)
Other:
- note added: "I2C 0x3c"
- note added: "Measured:\n<0.5mA\n"
- note added: "Oled display"
- note added: "Spec:\n1-75mA, 20mA avg\nMeasured:\n4.3mA at idle, 60mA at readout"
- note added: "U5 - BMP280 should allow to set i2c address\nby connecting SDO to either gnd or Vcc"
- note removed: "Spec:\n1-75mA, 20mA avg\nMeasured:\n<5mA at idle, 60mA at readout"
Changed lines of the file:
@@
 P 13800 8450
 F 0 "U5" H 13350 8100 50  0000 R CNN
-F 1 "BME280" H 13600 8000 50  0000 R CNN
+F 1 "BMP280" H 13600 8000 50  0000 R CNN
 F 2 "Package_LGA:Bosch_LGA-8_2.5x2.5mm_P0.65mm_ClockwisePinNumbering" H 15300 8000 50  0001 C CNN
 F 3 "https://ae-bst.resource.bosch.com/media/_tech/media/datasheets/BST-BME280-DS002.pdf" H 13800 8250 50  0001 C CNN
@@
 Power\nConsumption
 Text Notes -4300 5250 0    44   ~ 0
-Spec:\n1-75mA, 20mA avg\nMeasured:\n<5mA at idle, 60mA at readout
+Spec:\n1-75mA, 20mA avg\nMeasured:\n4.3mA at idle, 60mA at readout
 Text Notes -2750 5150 0    44   ~ 0
 I2C 0xc2
@@
 Text Notes -3700 1600 0    118  ~ 0
 Bugs
+Text Notes -4300 5900 0    44   ~ 0
+Measured:\n<0.5mA\n
+Text Label 15300 7800 0    44   ~ 0
+BMP280_VCC
+Text Notes -5750 7000 2    118  ~ 0
+Oled display
+Text Notes -2750 6950 0    44   ~ 0
+I2C 0x3c
+Text Notes -3700 2150 0    44   ~ 0
+U5 - BMP280 should allow to set i2c address\nby connecting SDO to either gnd or Vcc
 $EndSCHEMATC
