File: KiCad/EnvSensor-v2/EnvSensor-v2.kicad_pcb (KiCad board)
At the start: 2 copper layers, 120 x 100 mm, 162 parts, among them J1 JTAG, J10 Conn_01x02, J2 Conn_01x02, J3 USB_B_Micro, J4 Conn_01x02, J5 Micro_SD_Card_Det, J6 Conn_01x02, J7 I2C, J8 HPMA115C0-003, J9 Conn_01x02, P1 USB_C_Plug_USB2.0, Q1 IRLML2502, Q2 Si3407DV, Q3 AUiRLR3110Z, Q4 AO6804A, SW1 SW_Push, SW2 Reset, SW3 SW_Push, SW4 SW_Push, SW5 SW_Push, SW6 Start, U1 STM32L451RCT6, U10 LTC3440, U11 MCP1826S-5.0, U12 MCP1825S-3.3, U13 ESP-12S, U2 E-Ink_Waveshare_4.2, U3 SCD30, U4 SCD40, U5 BME280, U6 AP9101CK, U7 MCP73843-4.2, U8 BME280-Module, U9 LM2735XMF, Y1 16Hz, Y2 32768/12.5pF

Commit message: pcb updates
Parts:
- C45: value 1u -> 100n
- Q3: value AUiRLR3110Z -> IRFR9024
- R17: value R -> 3k
- R18: value R -> 10k
- U5: value BME280 -> BMP280
Connections:
- net Net-(C20-Pad1) renamed /BMP280_VCC

Commit message: touchgfx introduced
Parts:
- Q3: value IRFR9024 -> ZXMP6A16K
Connections:
- net E_INK_CD renamed E_INK_DC

Commit message: More pcb work
Other:
- net class Default removed
- net class Power removed
- net class Thick removed
