File: KiCad/EnvSensor-v2/EnvSensor-v2.kicad_sch (KiCad schematic)
At the start: 163 parts

Commit message: Refactor
Parts:
- gave numbers to parts that had none: 158
Other:
- note added: "Vdd and Vss swapped in SD card"

Commit message: More pcb work
Other:
- note added: "Vdd and Vss swapped in SD card Q2 zonk!"
- note removed: "Vdd and Vss swapped in SD card"
Changed lines of the file:
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@@
     (effects (font (size 2.9972 2.9972)) (justify left bottom))
   )
-  (text "Vdd and Vss swapped in SD card" (at -93.98 64.77 0)
+  (text "Vdd and Vss swapped in SD card\nQ2 zonk!" (at -93.98 64.77 0)
     (effects (font (size 1.1176 1.1176)) (justify left bottom))
   )
