File: KiCad/EnvSensor-v2.1/EnvSensor-v2.1.kicad_sch (KiCad schematic)
At the start: 90 parts, among them J1 BattSense, J2 USB_B_Micro, J3 USB_C_Plug_USB2.0, J4 USB_C_Receptacle_USB2.0, J5 Conn_01x02, J6 Conn_01x02, Q1 AO6804A, Q2 IRLML2502, Q3 ZXMP6A16K, SW1 BATT_SWITCH, SW2 Start, U1 AP9101CK, U2 MCP1826S-5.0, U3 LM2735XMF, U4 MCP73843-4.2, U5 MCP1825S-3.3, U6 LTC3440

Commit message: poznan commit
Parts:
- removed C1: 10n, Capacitor_SMD:C_0805_2012Metric, symbol Device:C
- removed Q2: IRLML2502, Package_TO_SOT_SMD:SOT-23, symbol Transistor_FET:IRLML2060
- removed R1: 3k, Resistor_SMD:R_0805_2012Metric, symbol Device:R
- removed R3: 10k, Resistor_SMD:R_0603_1608Metric, symbol Device:R
- removed R5: 100k, Resistor_SMD:R_0603_1608Metric, symbol Device:R
- added C? (x2): 47u, Capacitor_SMD:C_1206_3216Metric, symbol Device:C
- added C? (x2): 22u, Capacitor_SMD:C_1206_3216Metric, symbol Device:C
- added C? (x4): 2u2, Capacitor_SMD:C_1206_3216Metric, symbol Device:C
- added D?: D_TVS, symbol Device:D_TVS
- added JP?: NO, Jumper:SolderJumper-2_P1.3mm_Open_RoundedPad1.0x1.5mm, symbol EnvSensor-v2-rescue:Jumper_NO_Small-Device
- added JP?: NC, Jumper:SolderJumper-2_P1.3mm_Bridged_RoundedPad1.0x1.5mm, symbol EnvSensor-v2-rescue:Jumper_NC_Small-Device
- added L?: 100-600R, symbol Device:L_Ferrite_Small
- added L?: 1u, Inductor_SMD:L_TDK_SLF10145, symbol Device:L
- added L?: 100-600, symbol Device:L_Ferrite_Small
- added Q?: IRLML2244, symbol Device:Q_PMOS_GSD
- added R?: 100R, symbol Device:R
- added R?: 12R5, symbol Device:R
- added R? (x2): 5R1, symbol Device:R
- added R?: 511k, Resistor_SMD:R_0805_2012Metric, symbol Device:R
- added R?: 91k, Resistor_SMD:R_0805_2012Metric, symbol Device:R
- added R?: 25R, symbol Device:R
- added R?: 3k3, Resistor_SMD:R_0805_2012Metric, symbol Device:R
- added R?: 50R, symbol Device:R
- added U?: TPS631000, symbol myLib:TPS631000
Connections:
- net +BATT: now also C?.1, L?.1; no longer C21.1, C22.1, C23.1, JP4.1, TS7.1, U6.7 (Vin), U6.8 (SHND/SS)
- net GND: now also J4.A1 (GND), J4.A12 (GND), J4.B1 (GND), J4.B12 (GND), C?.2, C?.2, C?.2, C?.2, C?.2, C?.2, C?.2, C?.2, D?.1 (A1), JP?.2, R?.1, R?.1, R?.2, R?.2, R?.2, R?.2, R?.2, R?.2, U?.7 (GND)
- net VBUS: now also J4.A4 (VBUS), J4.A9 (VBUS), J4.B4 (VBUS), J4.B9 (VBUS), D?.2 (A2), Q?.3 (D); no longer D1.2 (A)
- net at C3.1, D5.2 (A), D6.2 (A)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: now also Q?.2 (S); no longer D1.1 (K)
- net 3V3_NOT_REG: now reaches C16.1, C17.1, C18.1, C19.1, D8.1 (K), R14.1, TS6.1, U6.6 (Vout)
- net 3V3_NOT_REG: now also C?.1, C?.1, C?.1, L?.1, R?.2, U?.1 (Vout); no longer U5.1 (VI)
- net at J4.A5 (CC1): now also R?.1
- net at J4.B5 (CC2): now also R?.1
- new net: C?.1, L?.2, U5.1 (VI)
- new net: JP?.1, JP?.2, U?.6 (Mode)
- new net: L?.1, U?.3 (LX1)
- new net: L?.2, U?.2 (LX2)
- new net: R?.1, R?.2, U?.8 (FB)
- new net: Q?.1 (G), R?.2
- new net BATT_3V3_FILTER: C21.1, C22.1, C23.1, C?.1, C?.1, C?.1, JP4.1, JP?.1, L?.2, TS7.1, U6.7 (Vin), U6.8 (SHND/SS), U?.4 (Vin), U?.5 (EN)
- no-connect marks 9 -> 14
Other:
- note added: "3.3V Buck-Boost DC/DC Converter with TPS631000"
- note added: "Ctimer=C14+C15 Tfast_charge=Ctimer/100n * 1.5h Telapsed=Ctimer/100n * 3h"
- note added: "Dummy Load"
- note added: "Tin=1*22u"
- note added: "Tout=1*47u"
- note added: "U=3.3V U=5V R=100R 33mA / 109mW 50mA / 250mW R=50R 66mA / 218mW 100mA / 500mW R=25R 132mA / 436mW 200mA / 1W R=12.5R 264mA / 871mW 400mA / 2W"
- note removed: "Battery Voltage Sense"
- note removed: "Ctimer=? Tfast_charge=Ctimer/100n * 1.5h Telapsed=Ctimer/100n * 3h"
- note removed: "Vmax=4.3V Vref=3.3V R17+R18=4.3V/3.3V*10k =13k"
- moved on the sheet: B1, B2, B3, C10, C11, C12, C13, C14, C15, C16, C17, C18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

Commit message: pcb started
Parts:
- removed J3: USB_C_Plug_USB2.0, JPConnectors:USB_C_Receptacle_Adam_Tech, symbol EnvSensor-v2-rescue:USB_C_Plug_USB2.0-Connector
- added C1, C2: 4n7, Capacitor_SMD:C_0805_2012Metric, symbol Device:C
- added C26: 1u, Capacitor_SMD:C_0805_2012Metric, symbol Device:C
- added C27: 47n, Capacitor_SMD:C_0805_2012Metric, symbol Device:C
- added C33, C35, C40, C41: 2u2, Capacitor_SMD:C_1206_3216Metric, symbol Device:C
- added C36: 22n, Capacitor_SMD:C_0805_2012Metric, symbol Device:C
- added C42: 100n, Capacitor_SMD:C_0603_1608Metric, symbol Device:C
- added D10: INPUT POWER LED, LED_THT:LED_D3.0mm_Horizontal_O3.81mm_Z6.0mm, symbol Device:LED
- added D11, D9: POWER LED, LED_SMD:LED_0805_2012Metric, symbol Device:LED
- added D12: CHARGE LED, LED_THT:LED_D3.0mm_Horizontal_O3.81mm_Z6.0mm, symbol Device:LED
- added D13: 3.3V POWER LED, LED_THT:LED_D3.0mm_Horizontal_O3.81mm_Z6.0mm, symbol Device:LED
- added D14: 5V POWER LED, LED_THT:LED_D3.0mm_Horizontal_O3.81mm_Z6.0mm, symbol Device:LED
- added J6: POWER_OUTPUT, Connector_PinHeader_2.54mm:PinHeader_2x07_P2.54mm_Vertical, symbol Connector_Generic:Conn_02x07_Odd_Even
- added L6, L7: 100-600R, Inductor_SMD:L_0805_2012Metric, symbol Device:L_Ferrite_Small
- added R16: 73k2, Resistor_SMD:R_0805_2012Metric, symbol Device:R
- added R23: 4R7, Resistor_SMD:R_0805_2012Metric, symbol Device:R
- added R24: DNP, Resistor_SMD:R_1206_3216Metric, symbol Device:R
- added R25: 0R05, Resistor_SMD:R_1206_3216Metric, symbol Device:R
- added R26: 10k, Resistor_SMD:R_0603_1608Metric, symbol Device:R
- added R27, R28, R29, R30: 3k3, Resistor_SMD:R_0805_2012Metric, symbol Device:R
- added TP1, TP2, TP3, TP4, TP5, TP6: TestPoint, TestPoint:TestPoint_Pad_D1.5mm, symbol Connector:TestPoint
- added U7: LTC4052, Package_SO:MSOP-8_3x3mm_P0.65mm, symbol myLib:LTC4052
- D1: renamed from D?; value D_TVS -> PESD5V0V1BA; footprint (none) -> Diode_SMD:D_SOD-323
- D2: renamed from D7; value PMEG2010AEJ -> DNP (PMEG2010AEJ)
- D3: renamed from D8; value PMEG3020BER -> DNP (PMEG3020BER)
- L2, L3: renamed from L?; footprint (none) -> Inductor_SMD:L_0805_2012Metric
- Q2: renamed from Q?; footprint (none) -> Package_TO_SOT_SMD:SOT-23
- R1, R2: renamed from R?; value 5R1 -> 5k1; footprint (none) -> Resistor_SMD:R_0805_2012Metric
- R17: renamed from R?; value 511k -> 120k
- R20: renamed from R?; value 91k -> 30k
- R3, R4, R5, R6: renamed from R?; footprint (none) -> Resistor_SMD:R_2512_6332Metric
- TS1: renamed from TS4; footprint TestPoint:TestPoint_THTPad_D1.5mm_Drill0.7mm -> TestPoint:TestPoint_Pad_D1.5mm
- TS2: renamed from TS5; footprint TestPoint:TestPoint_THTPad_D1.5mm_Drill0.7mm -> TestPoint:TestPoint_Pad_D1.5mm
- TS3: renamed from TS6; footprint TestPoint:TestPoint_THTPad_D1.5mm_Drill0.7mm -> TestPoint:TestPoint_Pad_D1.5mm
- TS4: renamed from TS7; footprint TestPoint:TestPoint_THTPad_D1.5mm_Drill0.7mm -> TestPoint:TestPoint_Pad_D1.5mm
- TS5: renamed from TS1; footprint TestPoint:TestPoint_THTPad_D1.5mm_Drill0.7mm -> TestPoint:TestPoint_Pad_D1.5mm
- TS6: renamed from TS2; footprint TestPoint:TestPoint_THTPad_D1.5mm_Drill0.7mm -> TestPoint:TestPoint_Pad_D1.5mm
- TS7: renamed from TS3; footprint TestPoint:TestPoint_THTPad_D1.5mm_Drill0.7mm -> TestPoint:TestPoint_Pad_D1.5mm
- U4: renamed from U?; footprint (none) -> Package_TO_SOT_SMD:SOT-23-8
- gave numbers to parts that had none: 12
- renumbered C23 to C10, C24 to C11, C25 to C12, C20 to C15, C3 to C18, C4 to C23, C14 to C24, C15 to C25, C5 to C28, C6 to C29, C16 to C3, C7 to C30, C8 to C31, C9 to C32, C10 to C34, C11 to C37, C12 to C38, C13 to C39, C17 to C4, C18 to C5, C19 to C6, C2 to C7, C21 to C8, C22 to C9, D2 to D15, D1 to D4, D3 to D5, D4 to D6, D5 to D7, D6 to D8, J2 to J1, J4 to J2, J1 to J3, J6 to J4, JP4 to JP2, JP5 to JP3, JP3 to JP4, JP2 to JP7, L2 to L1, L1 to L5, R15 to R10, R16 to R11, R17 to R12, R18 to R13, R19 to R14, R6 to R15, R8 to R19, R11 to R21, R12 to R22, R7 to R31, R9 to R32, R10 to R33, R13 to R34, R2 to R7, R14 to R8, R4 to R9, U6 to U1, U1 to U2, U5 to U3, U4 to U5, U2 to U6, U3 to U8
Connections:
- net +3V3: now also D13.2 (A), J6.7 (Pin_7), J6.9 (Pin_9), TP1.1
- net +5V: now also D14.2 (A), J6.3 (Pin_3), J6.5 (Pin_5), TP2.1
- net +BATT: now also C40.1, J6.11 (Pin_11), L7.1, U7.8 (BAT); no longer C37.1, C38.1, C39.1, L5.1, TS7.1, U8.5 (VIN)
- net 3V3_NOT_REG: now also R16.2; no longer R17.2
- net GND: now also C1.2, C2.2, C26.2, C33.2, C35.2, C36.2, C40.2, C41.2, C42.2, J6.10 (Pin_10), J6.12 (Pin_12), J6.14 (Pin_14), J6.2 (Pin_2), J6.4 (Pin_4), J6.6 (Pin_6), J6.8 (Pin_8), R29.1, R30.1, U7.4 (GND)
- net POWER_5V_ENABLE: now also J6.13 (Pin_13)
- net VBUS: now also D10.2 (A), D11.2 (A), D12.2 (A), D9.2 (A), J6.1 (Pin_1), R23.1, R24.1, R25.1, R26.1, U7.3 (VIN)
- net at J1.6 (Shield): now also C1.1
- net 3V3_REG: now reaches C15.1, J4.1 (Pin_1), JP4.1, U3.3 (VO)
- net at C28.1, C29.1, C30.1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: now also C33.1, L6.1; no longer U6.1 (VI)
- net 3V3_LTC_SW1: now reaches D2.1 (K), L1.1, TS1.1, U1.3 (SW1)
- net 3V3_LTC_SW2: now reaches D3.2 (A), L1.2, TS2.1, U1.4 (SW2)
- net 3V3_LTC_FB: now reaches R10.2, R11.1, R8.2, U1.9 (FB)
- net at R3.1: now also TP3.1
- net at R6.1: now also TP6.1
- net at J2.S1 (SHIELD): now also C2.1
- net at R5.1: now also TP5.1
- net at R4.1: now also TP4.1
- new net: C37.1, C38.1, C39.1, C41.1, L5.1, L7.2, TS7.1, U8.5 (VIN)
- new net: C35.1, L6.2, U6.1 (VI)
- new net: C27.1, R26.2
- new net: R24.2, R25.2, U7.1 (SENSE)
- new net: R27.1, U7.2 (ACPR)
- new net: C42.1, U7.5 (TIMER)
- new net: R28.1, U7.6 (CHRG)
- new net: C27.2, C36.1, U7.7 (GATE)
- new net: D11.1 (K), D12.1 (K), R28.2
- new net: R16.1, R17.2
- new net: D13.1 (K), R29.2
- new net: C26.1, R23.2
- new net: D10.1 (K), D9.1 (K), R27.2
- new net: D14.1 (K), R30.2
- no-connect marks 14 -> 7
Other:
- note added: "4.5V <= Vin <= 10V Current Limited Power Supply Only! Imax=2 * Power Supply Current Limit Imax=105mV/(Rsense+10mR) Imax=105mV/(50mR+10mR)=1.75A Psense=Rsense*Icharge^2 Psense=0.11W"
- note added: "Cin=1*22u"
- note added: "Cout=1*47u"
- note added: "Ctimer=Cx+Cy Ttimer=Ctimer/100n * 3h"
- note added: "Impulse Battery Charger"
- note added: "Li-Ion 1 cell 4.2V"
- note added: "Linear Battery Charger"
- note added: "P=Icharge^2*Rds(on) P=1.5A^2*0.35R=0.8W DeltaT=35deg/W*0.8W=26deg"
- note added: "Rosc=60k fosc=1MHz"
- note added: "Vdropout = 210mV typ / 350mV max Vin(min)=3.3V + 0.35V=3.65V"
- note added: "Vfb=500mV Rbottom <= 100k Rtop=Rbottom*(Vout/Vfb-1) Rtop=30k*6.3=189k Rtop=47k*6.3=296k1 Rtop=68k*6.3=428k4"
- note added: "Vout=Vfb*((Rtop+Rbottom)/Rbottom) Vout=0V5*((120k+73k2+30k)/30k)=3.72V Vout=0V5*((220k+73k2+47k)/47k)=3.62V Iout(max)=1A5"
- note removed: "Battery Charger"
- note removed: "Tin=1*22u"
- note removed: "Tout=1*47u"
- title: (none) -> Environmental Sensor Power Supply
- moved on the sheet: B1, B2, B3, C10, C11, C12, C13, C14, C15, C16, C17, C18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

Commit message: More pcb work
Parts:
- removed C2: 4n7, Capacitor_SMD:C_0805_2012Metric, symbol Device:C
- removed D10: INPUT POWER LED, LED_THT:LED_D3.0mm_Horizontal_O3.81mm_Z6.0mm, symbol Device:LED
- removed D11, D9: POWER LED, LED_SMD:LED_0805_2012Metric, symbol Device:LED
- removed D12: CHARGE LED, LED_THT:LED_D3.0mm_Horizontal_O3.81mm_Z6.0mm, symbol Device:LED
- removed D4: PMEG3020BER, Diode_SMD:D_SOD-123, symbol Device:D
- removed D8: CHARGE LED - Red, LED_THT:LED_D3.0mm_Horizontal_O3.81mm_Z6.0mm, symbol Device:LED
- removed R27, R28: 3k3, Resistor_SMD:R_0805_2012Metric, symbol Device:R
- added C43: 100n, Capacitor_SMD:C_0603_1608Metric, symbol Device:C
- added D4: POWER LED, LED_SMD:LED_0805_2012Metric, symbol Device:LED
- added F1, F2, F3: 0ZCJ0110FF2E, Fuse:Fuse_1206_3216Metric, symbol Device:Fuse
- added JP8, JP9: NO, Jumper:SolderJumper-2_P1.3mm_Open_RoundedPad1.0x1.5mm, symbol EnvSensor-v2-rescue:Jumper_NO_Small-Device
- C13, C14, C16, C17, C33, C35, C40, C41: footprint Capacitor_SMD:C_1206_3216Metric -> Capacitor_SMD:C_0805_2012Metric
- D13, D14: footprint LED_THT:LED_D3.0mm_Horizontal_O3.81mm_Z6.0mm -> LED_SMD:LED_0805_2012Metric
- D6: value POWER LED -> POWER LED (Red)
- D7: value CHARGE LED - Red -> CHARGE LED (Red); footprint LED_SMD:LED_0805_2012Metric -> LED_THT:LED_D3.0mm_Horizontal_O3.81mm_Z6.0mm
- U4: footprint Package_TO_SOT_SMD:SOT-23-8 -> JPPackages:SOT-5x3
Connections:
- net +BATT: now also R7.1
- net -BATT: now also F1.2, F2.2, F3.2; no longer B1.2 (-), B2.2 (-), B3.2 (-)
- net GND: now also C43.2, JP8.2; no longer R19.1
- net VBUS: now also D7.2 (A), D4.2 (A)
- net L_CHRG_SENSE: now reaches Q3.3 (S), R15.1, U5.1 (SENSE)
- net L_CHRG_POWER: now reaches C18.1, Q2.2 (S), R15.2, R22.2, U5.2 (VDD)
- net L_CHRG_POWER: no longer D7.2 (A)
- net at R21.2: now also D7.1 (K), D4.1 (K); no longer U5.3 (STAT1)
- net L_CHRG_EN: now reaches R22.1, U5.4 (EN)
- net L_CHRG_TIMER: now reaches C24.1, C25.1, U5.5 (TIMER)
- net L_CHRG_DRV: now reaches Q3.1 (G), U5.8 (DRV)
- net PROT_VDD: now reaches C7.1, R7.2, U2.2 (VDD)
- net BATT_SW: now reaches J3.1 (Pin_1), JP1.1, SW1.2 (B)
- net BATT_SW: no longer R7.1
- net CHRG_CHRG: now reaches R21.1
- net CHRG_CHRG: now also U5.3 (STAT1), U7.6 (CHRG); no longer D7.1 (K)
- net USB_SHIELD: now reaches C1.1, J1.6 (Shield)
- net USB_SHIELD: now also J2.S1 (SHIELD)
- net 5V_FB: now reaches C28.2, R31.2, R33.1, U8.3 (FB)
- net 5V_IN: now reaches C37.1, C38.1, C39.1, C41.1, L5.1, L7.2, TS7.1, U8.5 (VIN)
- net 5V_NOT_REG: now reaches C28.1, C29.1, C30.1, C31.1, C32.1, C33.1, D15.1 (K), L6.1, R31.1, TS6.1
- net 3V3_LTC_Rt: now reaches R12.1, U1.1 (Rt)
- net 3V3_LTC_VC: now reaches C11.2, C12.2, U1.10 (Vc)
- net 3V3_LTC_MODE: now reaches JP2.2, JP3.1, U1.2 (MODE/SYNC)
- net PROT_DRAIN: now reaches Q1.2 (D2), Q1.5 (D2)
- net 5V_FILTERED: now reaches C35.1, L6.2, U6.1 (VI)
- net 3V3_FILTER: now reaches C14.1, L2.2, U3.1 (VI)
- net 3V3_TSP_MODE: now reaches JP5.2, JP6.1, U4.6 (Mode)
- net I_CHRG_SENSE: now reaches R24.2, R25.2, U7.1 (SENSE)
- net CHRG_ACPR: now reaches U7.2 (ACPR)
- net CHRG_ACPR: now also JP9.2
- net I_CHRG_TIMER: now reaches C42.1, U7.5 (TIMER)
- net I_CHRG_TIMER: now also C43.1
- net I_CHRG_GATE: now reaches C27.2, C36.1, U7.7 (GATE)
- net 3V3_TSP_LX1: now reaches L4.1, U4.3 (LX1)
- net 3V3_TSP_LX2: now reaches L4.2, U4.2 (LX2)
- net 3V3_TSP_FB: now reaches R17.1, R20.2, U4.8 (FB)
- new net: JP8.1, JP9.1, R19.1
- new net BATT1-: B1.2 (-), F1.1
- new net BATT2-: B2.2 (-), F2.1
- new net BATT3-: B3.2 (-), F3.1
Other:
- note added: "Connect to GND for MCP73843 Connect to CHRG_ACPR for LTC4052"
- note added: "Imax=500mA I=110mA | 250mA P=0.4V*110mA | 0.4V*250mA P=44mW | 100mW"
- note added: "Polimer PTC 1.1A"
- note removed: "Imax=110mA | 250mA Pmax=0.4V*110mA | 0.4V*250mA Pmax=44mW | 100mW"
- moved on the sheet: B1, B2, B3, C10, C11, C12, C13, C14, C15, C16, C17, C19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
