File: KiCad/EnvSensor-v2.1/EnvSensor-v2.1.kicad_sch (KiCad schematic)
At the start: 141 parts, among them J1 USB_B_Micro, J2 USB_C_Receptacle_USB2.0, J3 BattSense, J4 Conn_01x02, J5 Conn_01x02, J6 POWER_OUTPUT, Q1 AO6804A, Q2 IRLML2244, Q3 ZXMP6A16K, SW1 BATT_SWITCH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

Commit message: pcb
Connections:
- net +3V3: now also J6.1 (Pin_1), J6.3 (Pin_3); no longer J6.5 (Pin_5), J6.7 (Pin_7)
- net +5V: now also J6.5 (Pin_5), J6.7 (Pin_7); no longer J6.1 (Pin_1), J6.3 (Pin_3)
Changed lines of the file:
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@@
     (pin "1")
   )
-  (symbol (lib_id "power:+5V") (at 508 299.72 0) (unit 1)
-    (in_bom yes) (on_board yes)
-    (property "Reference" "#PWR058" (id 0) (at 508 303.53 0)
-      (effects (font (size 1.27 1.27)) hide)
-    )
-    (property "Value" "+5V" (id 1) (at 508.381 295.3258 0))
-    (property "Footprint" "" (id 2) (at 508 299.72 0)
-      (effects (font (size 1.27 1.27)) hide)
-    )
-    (property "Datasheet" "" (id 3) (at 508 299.72 0)
+  (symbol (lib_id "power:+5V") (at 502.92 304.8 0) (unit 1)
+    (in_bom yes) (on_board yes)
+    (property "Reference" "#PWR058" (id 0) (at 502.92 308.61 0)
+      (effects (font (size 1.27 1.27)) hide)
+    )
+    (property "Value" "+5V" (id 1) (at 503.301 300.4058 0))
+    (property "Footprint" "" (id 2) (at 502.92 304.8 0)
+      (effects (font (size 1.27 1.27)) hide)
+    )
+    (property "Datasheet" "" (id 3) (at 502.92 304.8 0)
       (effects (font (size 1.27 1.27)) hide)
     )
@@
     (pin "2")
   )
-  (symbol (lib_id "EnvSensor-v2-rescue:+3.3V-power") (at 502.92 304.8 0) (unit 1)
-    (in_bom yes) (on_board yes)
-    (property "Reference" "#PWR062" (id 0) (at 502.92 308.61 0)
-      (effects (font (size 1.27 1.27)) hide)
-    )
-    (property "Value" "+3.3V" (id 1) (at 503.301 300.4058 0))
-    (property "Footprint" "" (id 2) (at 502.92 304.8 0)
-      (effects (font (size 1.27 1.27)) hide)
-    )
-    (property "Datasheet" "" (id 3) (at 502.92 304.8 0)
-      (effects (font (size 1.27 1.27)) hide)
-    )
+  (symbol (lib_id "EnvSensor-v2-rescue:+3.3V-power") (at 508 299.72 0) (unit 1)
+    (in_bom yes) (on_board yes)
+    (property "Reference" "#PWR062" (id 0) (at 508 303.53 0)
+      (effects (font (size 1.27 1.27)) hide)
+    )
+    (property "Value" "+3.3V" (id 1) (at 508.381 295.3258 0))
+    (property "Footprint" "" (id 2) (at 508 299.72 0)
+      (effects (font (size 1.27 1.27)) hide)
+    )
+    (property "Datasheet" "" (id 3) (at 508 299.72 0)
+      (effects (font (size 1.27 1.27)) hide)
+    )

Commit message: Upgrade to STM32CubeIDE 1.12
Connections:
- net BATT_BARE: now also SW1.2 (B); no longer SW1.1 (A)
- net BATT_SW: now also SW1.1 (A); no longer SW1.2 (B)
Other:
- moved on the sheet: SW1
Changed lines of the file:
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@@
     (pin "S1")
   )
-  (symbol (lib_id "Switch:SW_SPST") (at 47.625 127 0) (unit 1)
+  (symbol (lib_id "Switch:SW_SPST") (at 47.625 127 180) (unit 1)
     (in_bom yes) (on_board yes)
-    (property "Reference" "SW1" (id 0) (at 47.625 121.6492 0))
-    (property "Value" "BATT_SWITCH" (id 1) (at 47.625 124.1861 0))
+    (property "Reference" "SW1" (id 0) (at 47.625 132.3508 0))
+    (property "Value" "BATT_SWITCH" (id 1) (at 47.625 129.8139 0))
     (property "Footprint" "Button_Switch_THT:SW_Tactile_SPST_Angled_PTS645Vx31-2LFS" (id 2) (at 47.625 127 0)
       (effects (font (size 1.27 1.27)) hide)

Commit message: Final PCB work
Connections:
- net +BATT: now also J6.11 (Pin_11); no longer J6.9 (Pin_9)
- net POWER_5V_ENABLE: now also J6.9 (Pin_9); no longer J6.13 (Pin_13)
- net VBUS: now also J6.13 (Pin_13); no longer J6.11 (Pin_11)
- net T100: now reaches R3.1, TP3.1
- net T12.5: now reaches R6.1, TP6.1
- net T25: now reaches R5.1, TP5.1
- net T50: now reaches R4.1, TP4.1
Other:
- note added: "4.5V <= Vin <= 10V Current Limited Power Supply Only! Imax=2 * Power Supply Current Limit Imax=105mV/(Rsense+10mR) Imax=105mV/(50mR+10mR)=1.75A Icharge(max)=1.5A Psense=Rsense*Icharge^2 Psense=0.11W"
- note removed: "4.5V <= Vin <= 10V Current Limited Power Supply Only! Imax=2 * Power Supply Current Limit Imax=105mV/(Rsense+10mR) Imax=105mV/(50mR+10mR)=1.75A Psense=Rsense*Icharge^2 Psense=0.11W"
Changed lines of the file:
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@@
     (stroke (width 0) (type default) (color 0 0 0 0))
   )
-  (wire (pts (xy 497.84 314.96) (xy 511.81 314.96))
-    (stroke (width 0) (type default) (color 0 0 0 0))
-  )
   (wire (pts (xy 127 289.56) (xy 127 292.1))
     (stroke (width 0) (type default) (color 0 0 0 0))
@@
     (stroke (width 0) (type default) (color 0 0 0 0))
   )
-  (wire (pts (xy 497.84 312.42) (xy 497.84 314.96))
+  (wire (pts (xy 487.68 312.42) (xy 487.68 320.04))
     (stroke (width 0) (type default) (color 0 0 0 0))
   )
@@
     (stroke (width 0) (type default) (color 0 0 0 0))
   )
-  (wire (pts (xy 510.54 320.04) (xy 511.81 320.04))
-    (stroke (width 0) (type default) (color 0 0 0 0))
-  )
   (wire (pts (xy 311.15 299.72) (xy 311.15 298.45))
     (stroke (width 0) (type default) (color 0 0 0 0))
@@
     (stroke (width 0) (type default) (color 0 0 0 0))
   )
+  (wire (pts (xy 510.54 314.96) (xy 511.81 314.96))
+    (stroke (width 0) (type default) (color 0 0 0 0))
+  )
   (wire (pts (xy 292.735 292.1) (xy 292.735 293.37))
     (stroke (width 0) (type default) (color 0 0 0 0))
@@
     (stroke (width 0) (type default) (color 0 0 0 0))
   )
+  (wire (pts (xy 487.68 320.04) (xy 511.81 320.04))
+    (stroke (width 0) (type default) (color 0 0 0 0))
+  )
   (wire (pts (xy 355.6 128.27) (xy 355.6 129.54))
     (stroke (width 0) (type default) (color 0 0 0 0))
@@
     (stroke (width 0) (type default) (color 0 0 0 0))
   )
-  (wire (pts (xy 494.03 317.5) (xy 511.81 317.5))
+  (wire (pts (xy 491.49 317.5) (xy 511.81 317.5))
     (stroke (width 0) (type default) (color 0 0 0 0))
   )
-  (wire (pts (xy 494.03 313.69) (xy 494.03 317.5))
+  (wire (pts (xy 491.49 313.69) (xy 491.49 317.5))
     (stroke (width 0) (type default) (color 0 0 0 0))
   )
@@
     (effects (font (size 2.9972 2.9972)) (justify left bottom))
   )
-  (text "4.5V <= Vin <= 10V\nCurrent Limited Power Supply Only!\nImax=2 * Power Supply Current Limit\nImax=105mV/(Rsense+10mR)\nImax=105mV/(50mR+10mR)=1.75A\n\nPsense=Rsense*Icharge^2\nPsense=0.11W"
+  (text "4.5V <= Vin <= 10V\nCurrent Limited Power Supply Only!\nImax=2 * Power Supply Current Limit\nImax=105mV/(Rsense+10mR)\nImax=105mV/(50mR+10mR)=1.75A\n\nIcharge(max)=1.5A\n\nPsense=Rsense*Icharge^2\nPsense=0.11W"
     (at 135.89 274.32 0)
     (effects (font (size 1.1176 1.1176)) (justify left bottom))
@@
     (effects (font (size 1.27 1.27)) (justify left bottom))
   )
+  (label "T50" (at 254 54.61 0)
+    (effects (font (size 1.27 1.27)) (justify left bottom))
+  )
   (label "3V3_LTC_FB" (at 387.35 146.05 0)
     (effects (font (size 1.27 1.27)) (justify left bottom))
@@
     (effects (font (size 1.27 1.27)) (justify left bottom))
   )
+  (label "T100" (at 243.84 54.61 0)
+    (effects (font (size 1.27 1.27)) (justify left bottom))
+  )
   (label "BATT_3V3_FILTER" (at 307.975 142.24 0)
     (effects (font (size 1.27 1.27)) (justify left bottom))
@@
     (effects (font (size 1.27 1.27)) (justify left bottom))
   )
+  (label "T25" (at 264.16 54.61 0)
+    (effects (font (size 1.27 1.27)) (justify left bottom))
+  )
   (label "3V3_NOT_REG" (at 431.8 135.89 0)
     (effects (font (size 1.27 1.27)) (justify left bottom))
@@
     (effects (font (size 1.27 1.27)) (justify left bottom))
   )
+  (label "T12.5" (at 274.32 54.61 0)
+    (effects (font (size 1.27 1.27)) (justify left bottom))
+  )
   (label "5V_FILTERED" (at 400.685 281.94 0)
     (effects (font (size 1.27 1.27)) (justify left bottom))
@@
     (effects (font (size 1.27 1.27)) (justify left bottom))
   )
-  (global_label "POWER_5V_ENABLE" (shape input) (at 510.54 320.04 180) (fields_autoplaced)
+  (global_label "POWER_5V_ENABLE" (shape input) (at 510.54 314.96 180) (fields_autoplaced)
     (effects (font (size 1.1176 1.1176)) (justify right))
-    (property "Intersheet References" "${INTERSHEET_REFS}" (id 0) (at 34.29 219.71 0)
+    (property "Intersheet References" "${INTERSHEET_REFS}" (id 0) (at 34.29 214.63 0)
       (effects (font (size 1.27 1.27)) hide)
     )
@@
     (pin "2")
   )
-  (symbol (lib_id "power:+BATT") (at 497.84 312.42 0) (unit 1)
+  (symbol (lib_id "power:+BATT") (at 491.49 313.69 0) (unit 1)
     (in_bom yes) (on_board yes)
-    (property "Reference" "#PWR068" (id 0) (at 497.84 316.23 0)
+    (property "Reference" "#PWR068" (id 0) (at 491.49 317.5 0)
       (effects (font (size 1.27 1.27)) hide)
     )
-    (property "Value" "+BATT" (id 1) (at 498.221 309.1688 90)
+    (property "Value" "+BATT" (id 1) (at 491.871 310.4388 90)
       (effects (font (size 1.27 1.27)) (justify left))
     )
-    (property "Footprint" "" (id 2) (at 497.84 312.42 0)
+    (property "Footprint" "" (id 2) (at 491.49 313.69 0)
       (effects (font (size 1.27 1.27)) hide)
     )
-    (property "Datasheet" "" (id 3) (at 497.84 312.42 0)
+    (property "Datasheet" "" (id 3) (at 491.49 313.69 0)
       (effects (font (size 1.27 1.27)) hide)
     )
@@
     (pin "2")
   )
-  (symbol (lib_id "power:VBUS") (at 494.03 313.69 0) (unit 1)
+  (symbol (lib_id "power:VBUS") (at 487.68 312.42 0) (unit 1)
     (in_bom yes) (on_board yes)
-    (property "Reference" "#PWR057" (id 0) (at 494.03 317.5 0)
+    (property "Reference" "#PWR057" (id 0) (at 487.68 316.23 0)
       (effects (font (size 1.27 1.27)) hide)
     )
-    (property "Value" "VBUS" (id 1) (at 494.411 309.2958 0))
-    (property "Footprint" "" (id 2) (at 494.03 313.69 0)
+    (property "Value" "VBUS" (id 1) (at 488.061 308.0258 0))
+    (property "Footprint" "" (id 2) (at 487.68 312.42 0)
       (effects (font (size 1.27 1.27)) hide)
     )
-    (property "Datasheet" "" (id 3) (at 494.03 313.69 0)
+    (property "Datasheet" "" (id 3) (at 487.68 312.42 0)
       (effects (font (size 1.27 1.27)) hide)
     )
