File: KiCad/EnvSensor-v2.1/EnvSensor-v2.1.kicad_pcb (KiCad board)
At the start: 4 copper layers, 102 x 100 mm, 141 parts, among them J1 USB_B_Micro, J2 USB_C_Receptacle_USB2.0, J3 BattSense, J4 Conn_01x02, J5 Conn_01x02, J6 POWER_OUTPUT, Q1 AO6804A, Q2 IRLML2244, Q3 ZXMP6A16K, SW1 BATT_SWITCH, SW2 Start, U1 LTC3440, U2 AP9101CK, U3 MCP1825S-3.3, U4 TPS631000, U5 MCP73843-4.2, U6 MCP1826S-5.0, U7 LTC4052, U8 LM2735XMF

Commit message: Final PCB work
Parts:
- D13, D14, D4, D5, R29, R30: moved to B.Cu
- moved R3 77.4 mm to (116.0, 100.8), turned to 0 degrees
- moved R4 75.8 mm to (116.0, 96.8), turned to 0 degrees
- moved R5 74.4 mm to (116.0, 92.8), turned to 0 degrees
- moved R6 73.5 mm to (116.0, 88.8), turned to 0 degrees
- moved TP3 70.3 mm to (110.8, 100.8), turned to 0 degrees
- moved TP4 68.3 mm to (110.8, 96.8), turned to 0 degrees
- moved TP5 66.8 mm to (110.8, 92.8), turned to 0 degrees
- moved TP6 65.8 mm to (110.8, 88.8), turned to 0 degrees
- moved TP1 62.9 mm to (100.0, 90.0)
- moved TP2 54.8 mm to (100.0, 97.5)
- moved C16 22.0 mm to (43.0, 56.2), turned to -90 degrees
- moved L3 20.4 mm to (45.7, 55.2), turned to 0 degrees
- moved C17 17.0 mm to (48.5, 56.2), turned to -90 degrees
- moved R21 13.5 mm to (27.0, 76.2)
- moved D4 13.4 mm to (25.2, 76.2)
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Connections:
- net Net-(R3-Pad1) renamed /T100
- net Net-(R4-Pad1) renamed /T50
- net Net-(R5-Pad1) renamed /T25
- net Net-(R6-Pad1) renamed /T12.5
- J6 pad 11: VBUS -> +BATT
- J6 pad 13: POWER_5V_ENABLE -> VBUS
- J6 pad 9: +BATT -> POWER_5V_ENABLE
Routing:
- net +BATT: track 15.0 -> 194.0 mm, vias 0 -> 2
- net VBUS: track 54.9 -> 232.0 mm
- net /CHRG_CHRG: track 1.16 -> 86.0 mm, vias 0 -> 4
- net POWER_5V_ENABLE: track 0.09 -> 54.0 mm, vias 0 -> 3
- net /BATT_3V3_FILTER: track 14.6 -> 60.4 mm
- net /CHRG_ACPR: track 3.63 -> 39.2 mm
- net +3V3: track 3.02 -> 37.7 mm
- net GND: track 140.7 -> 160.3 mm, vias 59 -> 64
- net /5V_IN: track 3.82 -> 14.1 mm
- net +5V: track 14.3 -> 24.1 mm
- net /3V3_NOT_REG: track 75.4 -> 67.9 mm
- net /L_CHRG_SENSE: track 2.84 -> 5.69 mm
- net /T50: track 0.00 -> 2.29 mm
- net /T25: track 0.00 -> 2.25 mm
- net /T12.5: track 0.00 -> 2.25 mm
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Other:
- board text added: "100R"
- board text added: "12R5"
- board text added: "12R5 25R 50R 100R"
- board text added: "25R"
- board text added: "3V3 5V 264mA 400mA 132mA 200mA 66mA 100mA 33mA 50mA"
- board text added: "50R"
- board text added: "EnvSensor - Power Supply JP, 8.04.2023"
- board text added: "LTC"
- board text added: "MCP"
- board text added: "MCP1825S-3.3"
- board text added: "MCP1826S-5.0"
- board text removed: "aabb"
