File: KiCad/EnvSensor-v2.1/EnvSensor-v2.1.kicad_pcb (KiCad board)
At the start: 4 copper layers, 102 x 100 mm, 141 parts, among them J1 USB_B_Micro, J2 USB_C_Receptacle_USB2.0, J3 BattSense, J4 Conn_01x02, J5 Conn_01x02, J6 POWER_OUTPUT, Q1 AO6804A, Q2 IRLML2244, Q3 ZXMP6A16K, SW1 BATT_SWITCH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

Commit message: Main PCB work
Other:
- board text added: "3.3V"
- board text added: "3V3 5V 12R5 264mA 400mA 25R 132mA 200mA 50R 66mA 100mA 100R 33mA 50mA"
- board text added: "5V_EN"
- board text added: "BAT+"
- board text added: "USB"
- board text removed: "12R5 25R 50R 100R"
- board text removed: "3V3 5V 264mA 400mA 132mA 200mA 66mA 100mA 33mA 50mA"
