File: KiCad/EnvSensor-Main-v2.1/EnvSensor-Main-v2.1.kicad_sch (KiCad schematic)
At the start: 81 parts

Commit message: Main PCB work
Parts:
- added J6: POWER_INPUT, Connector_PinSocket_2.54mm:PinSocket_2x07_P2.54mm_Vertical, symbol Connector_Generic:Conn_02x07_Odd_Even
- J?: value JTAG -> SWD
- JP3: footprint (none) -> Jumper:SolderJumper-3_P1.3mm_Bridged12_RoundedPad1.0x1.5mm
Connections:
- net +3V3: now also J6.1 (Pin_1), J6.3 (Pin_3)
- net +5V: now also J6.5 (Pin_5), J6.7 (Pin_7)
- net GND: now also J6.10 (Pin_10), J6.12 (Pin_12), J6.14 (Pin_14), J6.2 (Pin_2), J6.4 (Pin_4), J6.6 (Pin_6), J6.8 (Pin_8)
- net POWER_5V_ENABLE: now also J6.9 (Pin_9)
- new net +BATT: J6.11 (Pin_11)
- new net VBUS: J6.13 (Pin_13)
Other:
- moved on the sheet: J?

Commit message: more pcb work
Connections:
- net LED_1: now also U?.10 (PC2); no longer U?.11 (PC3)
- net LED_2: now also U?.8 (PC0); no longer U?.10 (PC2)
- net LED_3: now also U?.11 (PC3); no longer U?.9 (PC1)
- net LED_4: now also U?.9 (PC1); no longer U?.8 (PC0)
Other:
- note added: "Particles sensor is energised even when 5v power is off"
Changed lines of the file:
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@@
+    (effects (font (size 1.1176 1.1176)) (justify left bottom))
+  )
+  (text "Particles sensor is energised even when 5v power is off"
+    (at -71.12 80.01 0)
     (effects (font (size 1.1176 1.1176)) (justify left bottom))
   )
@@
     )
   )
-  (global_label "LED_3" (shape input) (at 52.07 133.35 180) (fields_autoplaced)
+  (global_label "LED_3" (shape input) (at 52.07 138.43 180) (fields_autoplaced)
+    (effects (font (size 1.1176 1.1176)) (justify right))
+    (property "Intersheetrefs" "${INTERSHEET_REFS}" (at 45.1395 138.43 0)
+      (effects (font (size 1.27 1.27)) (justify right) hide)
+    )
+  )
+  (global_label "LED_4" (shape input) (at 52.07 133.35 180) (fields_autoplaced)
     (effects (font (size 1.1176 1.1176)) (justify right))
     (property "Intersheetrefs" "${INTERSHEET_REFS}" (at 45.1395 133.35 0)
-      (effects (font (size 1.27 1.27)) (justify right) hide)
-    )
-  )
-  (global_label "LED_4" (shape input) (at 52.07 130.81 180) (fields_autoplaced)
-    (effects (font (size 1.1176 1.1176)) (justify right))
-    (property "Intersheetrefs" "${INTERSHEET_REFS}" (at 45.1395 130.81 0)
       (effects (font (size 1.27 1.27)) (justify right) hide)
     )
@@
     )
   )
-  (global_label "LED_1" (shape input) (at 52.07 138.43 180) (fields_autoplaced)
-    (effects (font (size 1.1176 1.1176)) (justify right))
-    (property "Intersheetrefs" "${INTERSHEET_REFS}" (at 45.1395 138.43 0)
+  (global_label "LED_1" (shape input) (at 52.07 135.89 180) (fields_autoplaced)
+    (effects (font (size 1.1176 1.1176)) (justify right))
+    (property "Intersheetrefs" "${INTERSHEET_REFS}" (at 45.1395 135.89 0)
       (effects (font (size 1.27 1.27)) (justify right) hide)
     )
@@
     )
   )
-  (global_label "LED_2" (shape input) (at 52.07 135.89 180) (fields_autoplaced)
-    (effects (font (size 1.1176 1.1176)) (justify right))
-    (property "Intersheetrefs" "${INTERSHEET_REFS}" (at 45.1395 135.89 0)
-      (effects (font (size 1.27 1.27)) (justify right) hide)
-    )
+  (global_label "LED_2" (shape input) (at 52.07 130.81 180) (fields_autoplaced)
+    (effects (font (size 1.1176 1.1176)) (justify right))
+    (property "Intersheetrefs" "${INTERSHEET_REFS}" (at 45.1395 130.81 0)
+      (effects (font (size 1.27 1.27)) (justify right) hide)
+    )

Commit message: Main work done on PCB
Parts:
- added C45: 100n, Capacitor_SMD:C_0805_2012Metric, symbol Device:C
- added Q1: IRLML2502, Package_TO_SOT_SMD:SOT-23, symbol Transistor_FET:IRLML2060
- added R16: 100k, Resistor_SMD:R_0805_2012Metric, symbol Device:R
- added R17: 3k, Resistor_SMD:R_0805_2012Metric, symbol Device:R
- added R18: 10k, Resistor_SMD:R_0805_2012Metric, symbol Device:R
Connections:
- net +BATT: now also R17.1
- net BATTERY_MEASURE_ENABLE: now also U?.37 (PC6), Q1.1 (G), R16.1; no longer U?.57 (PB5)
- net BATTERY_MEASURE_INPUT: now also U?.14 (PA0), C45.1, R17.2, R18.1
- net GND: now also C45.2, Q1.2 (S), R16.2
- new net: Q1.3 (D), R18.2
Other:
- note added: "Battery Voltage Sense"
- note added: "Vmax=4.3V Vref=3.3V R17+R18=4.3V/3.3V*10k =13k"

Commit message: Refactor
Parts:
- Q?: symbol EnvSensor-v2-rescue:Si3407DV-myLib -> myLib:Si3407DV
Connections:
- net GND: now also J?.6 (VSS); no longer J?.4 (VDD)
- net SD_3V3: now also J?.4 (VDD), Q?.1 (D), Q?.2 (D), Q?.5 (D), Q?.6 (D); no longer J?.6 (VSS), Q?.4 (S)
- new net: J?.2 (Pin_2), JP?.2, Q?.4 (S), R?.1
Other:
- moved on the sheet: Q?, R?
