File: KiCad/EnvSensor-Main-v2.1/EnvSensor-Main-v2.1.kicad_sch (KiCad schematic)
At the start: 92 parts, among them J6 POWER_INPUT, Q1 IRLML2502

Commit message: Bore moving swd and i2c
Connections:
- net LED_1: now also U?.11 (PC3); no longer U?.10 (PC2)
- net LED_2: now also U?.10 (PC2); no longer U?.8 (PC0)
- net LED_3: now also U?.9 (PC1); no longer U?.11 (PC3)
- net LED_4: now also U?.8 (PC0); no longer U?.9 (PC1)
Changed lines of the file:
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@@
     )
   )
-  (global_label "LED_3" (shape input) (at 52.07 138.43 180) (fields_autoplaced)
+  (global_label "LED_1" (shape input) (at 52.07 138.43 180) (fields_autoplaced)
     (effects (font (size 1.1176 1.1176)) (justify right))
-    (property "Intersheetrefs" "${INTERSHEET_REFS}" (at 45.1395 138.43 0)
+    (property "Intersheetrefs" "${INTERSHEET_REFS}" (at 44.494 138.43 0)
       (effects (font (size 1.27 1.27)) (justify right) hide)
     )
   )
-  (global_label "LED_4" (shape input) (at 52.07 133.35 180) (fields_autoplaced)
+  (global_label "LED_3" (shape input) (at 52.07 133.35 180) (fields_autoplaced)
     (effects (font (size 1.1176 1.1176)) (justify right))
-    (property "Intersheetrefs" "${INTERSHEET_REFS}" (at 45.1395 133.35 0)
+    (property "Intersheetrefs" "${INTERSHEET_REFS}" (at 44.494 133.35 0)
       (effects (font (size 1.27 1.27)) (justify right) hide)
     )
@@
     )
   )
-  (global_label "LED_1" (shape input) (at 52.07 135.89 180) (fields_autoplaced)
+  (global_label "LED_2" (shape input) (at 52.07 135.89 180) (fields_autoplaced)
     (effects (font (size 1.1176 1.1176)) (justify right))
-    (property "Intersheetrefs" "${INTERSHEET_REFS}" (at 45.1395 135.89 0)
+    (property "Intersheetrefs" "${INTERSHEET_REFS}" (at 44.494 135.89 0)
       (effects (font (size 1.27 1.27)) (justify right) hide)
     )
@@
     )
   )
-  (global_label "LED_2" (shape input) (at 52.07 130.81 180) (fields_autoplaced)
+  (global_label "LED_4" (shape input) (at 52.07 130.81 180) (fields_autoplaced)
     (effects (font (size 1.1176 1.1176)) (justify right))
-    (property "Intersheetrefs" "${INTERSHEET_REFS}" (at 45.1395 130.81 0)
+    (property "Intersheetrefs" "${INTERSHEET_REFS}" (at 44.494 130.81 0)
       (effects (font (size 1.27 1.27)) (justify right) hide)
     )

Commit message: Before moving i2c tracks
Parts:
- J?: footprint Connector_PinSocket_2.54mm:PinSocket_1x04_P2.54mm_Horizontal -> JPConnectors:PinSocket_1x04_P2.54mm_Horizontal_SMD
Changed lines of the file:
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@@
       (effects (font (size 1.27 1.27)) (justify left))
     )
-    (property "Footprint" "Connector_PinSocket_2.54mm:PinSocket_1x04_P2.54mm_Horizontal" (at 96.52 219.71 0)
+    (property "Footprint" "JPConnectors:PinSocket_1x04_P2.54mm_Horizontal_SMD" (at 96.52 219.71 0)
       (effects (font (size 1.27 1.27)) hide)
     )
