File: KiCad/EnvSensor-Main-v2.1/EnvSensor-Main-v2.1.kicad_pcb (KiCad board)
At the start: 4 copper layers, 102 x 100 mm, 82 parts, among them J1 Conn_01x02, J2 Conn_01x02, J3 HPMA115C0-003, J4 Conn_01x02, J5 Micro_SD_Card_Det, J6 SWD, J7 I2C, J8 POWER_INPUT, Q1 Si3407DV, SW1 Reset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

Commit message: more pcb work
Parts:
- moved R13 25.6 mm to (47.2, 68.8)
- moved R17 25.4 mm to (47.2, 67.5)
- moved C21 25.3 mm to (47.2, 66.2)
- moved R12 24.7 mm to (43.9, 68.8)
- moved R16 24.6 mm to (43.9, 67.5)
- moved C20 24.4 mm to (43.9, 66.2)
- moved R11 24.0 mm to (40.7, 68.8)
- moved R15 23.8 mm to (40.7, 67.5)
- moved C19 23.7 mm to (40.7, 66.2)
- moved R10 23.4 mm to (37.4, 68.7)
- moved R14 23.2 mm to (37.4, 67.5)
- moved C18 23.1 mm to (37.4, 66.2)
- moved JP1 21.6 mm to (97.2, 87.2), turned to 180 degrees
- moved J2 16.1 mm to (94.0, 49.6)
- moved JP2 15.7 mm to (92.0, 50.8)
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Connections:
- U5 pad 10: LED_2 -> LED_1
- U5 pad 11: LED_1 -> LED_3
- U5 pad 8: LED_4 -> LED_2
- U5 pad 9: LED_3 -> LED_4
Routing:
- net +3V3: track 15.4 -> 345.9 mm, vias 0 -> 16
- net SDA: track 0.00 -> 155.6 mm, vias 0 -> 1
- net SCL: track 0.00 -> 152.5 mm, vias 0 -> 2
- net +5V: track 0.00 -> 144.0 mm, vias 0 -> 4
- net POWER_5V_ENABLE: track 0.00 -> 92.6 mm, vias 0 -> 3
- net WIFI_RESET: track 0.00 -> 79.4 mm, vias 0 -> 1
- net WIFI_ENABLE: track 0.00 -> 75.2 mm, vias 0 -> 1
- net NRST: track 0.00 -> 69.8 mm, vias 0 -> 4
- net Net-(R10-Pad2): track 7.96 -> 76.4 mm
- net WFI_TX: track 0.00 -> 67.3 mm, vias 0 -> 1
- net WIFI_RX: track 0.00 -> 65.7 mm, vias 0 -> 1
- net Net-(R11-Pad2): track 7.96 -> 66.3 mm
- net SCD30_READY: track 0.00 -> 57.2 mm
- net LED_3: track 37.3 -> 94.1 mm, vias 0 -> 2
- net Net-(R13-Pad2): track 7.96 -> 63.1 mm
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
Commit message: Main work done on PCB
Parts:
- added C22: 100n, Capacitor_SMD:C_0805_2012Metric, B.Cu at (46.0, 56.8)
- added Q2: IRLML2502, Package_TO_SOT_SMD:SOT-23, B.Cu at (40.8, 56.8)
- added R22: 3k, Resistor_SMD:R_0805_2012Metric, B.Cu at (44.8, 59.8)
- added R23: 10k, Resistor_SMD:R_0805_2012Metric, B.Cu at (44.0, 57.0)
- added R24: 100k, Resistor_SMD:R_0805_2012Metric, B.Cu at (40.2, 59.8)
- moved C11 0.75 mm to (41.5, 48.8)
- moved R8 0.41 mm to (84.3, 57.5)
Connections:
- U5 pad 14: unconnected-(U5-PA0-Pad14) -> BATTERY_MEASURE_INPUT
- U5 pad 37: unconnected-(U5-PC6-Pad37) -> BATTERY_MEASURE_ENABLE
- U5 pad 57: BATTERY_MEASURE_ENABLE -> unconnected-(U5-PB5-Pad57)
Routing:
- net +BATT: track 0.00 -> 79.9 mm, vias 0 -> 2
- net BATTERY_MEASURE_ENABLE: track 0.00 -> 14.6 mm, vias 0 -> 1
- net BATTERY_MEASURE_INPUT: track 0.00 -> 11.8 mm, vias 0 -> 1
- net GND: track 76.2 -> 80.6 mm, vias 43 -> 47
- net POWER_5V_ENABLE: track 92.6 -> 95.8 mm
- net Net-(Q2-D): track 0.00 -> 2.52 mm
- net MOSI: track 25.6 -> 27.7 mm
- net +5V: track 144.0 -> 142.6 mm
- net SDIO_DATA1: track 33.5 -> 34.4 mm
- net SDIO_DATA0: track 35.9 -> 36.7 mm
- net SWO: track 43.2 -> 43.9 mm
- net WIFI_RESET: track 79.4 -> 78.8 mm
- net NRST: track 69.8 -> 69.2 mm
Other:
- board text added: "STM32L451RCT6"

Commit message: Refactor
Parts:
- JP1: moved to F.Cu
- moved JP4 6.74 mm to (37.8, 81.1), turned to -90 degrees
- moved R2 4.01 mm to (44.2, 80.5), turned to 0 degrees
- moved C10 3.62 mm to (73.2, 38.5)
- moved J4 2.23 mm to (39.8, 79.7), turned to 0 degrees
- moved JP1 0.15 mm to (97.0, 87.2)
- moved Q1 0.09 mm to (44.2, 83.2), turned to 180 degrees
- turned C14 to -90 degrees
- turned C15 to -90 degrees
Connections:
- J5 pad 4: GND -> /SD_3V3
- J5 pad 6: /SD_3V3 -> GND
- Q1 pad 1: Net-(J4-Pin_2) -> /SD_3V3
- Q1 pad 2: Net-(J4-Pin_2) -> /SD_3V3
- Q1 pad 4: /SD_3V3 -> Net-(J4-Pin_2)
- Q1 pad 5: Net-(J4-Pin_2) -> /SD_3V3
- Q1 pad 6: Net-(J4-Pin_2) -> /SD_3V3
Routing:
- net /SD_3V3: track 25.9 -> 32.6 mm
- net /VBAT: track 19.4 -> 23.1 mm
- net Net-(J4-Pin_2): track 11.1 -> 7.46 mm
- net SDIO_POWER_ENABLE: track 49.5 -> 46.2 mm
- net GND: track 80.6 -> 79.3 mm, vias 47 -> 46
- net SDIO_DATA0: track 36.7 -> 35.7 mm
- net WIFI_RESET: track 78.8 -> 77.9 mm
- net SDIO_DATA1: track 34.4 -> 33.5 mm
- net POWER_5V_ENABLE: track 95.8 -> 95.2 mm

Commit message: More pcb work
Routing:
- net +3V3: track 345.3 -> 349.7 mm
- net SWO: track 43.9 -> 46.4 mm
- net MOSI: track 27.7 -> 25.7 mm
- net Net-(R11-Pad2): track 66.3 -> 64.5 mm
- net Net-(R10-Pad2): track 76.4 -> 74.7 mm
- net Net-(R12-Pad2): track 61.2 -> 59.6 mm
- net Net-(R13-Pad2): track 63.1 -> 61.7 mm
- net WFI_TX: track 67.3 -> 66.0 mm
- net SCD30_READY: track 57.2 -> 57.9 mm
- net SWCLK: track 46.0 -> 46.6 mm
- net LED_4: track 96.7 -> 97.4 mm
- net WIFI_RESET: track 77.9 -> 78.5 mm
- net POWER_5V_ENABLE: track 95.2 -> 94.6 mm
- net SDIO_DETECT: track 52.2 -> 52.8 mm
- net SWDIO: track 48.1 -> 48.7 mm
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
Commit message: PCB work
Parts:
- moved R8 3.75 mm to (88.1, 57.5)
- moved R9 3.75 mm to (84.2, 57.5)
- moved C3 1.04 mm to (59.5, 53.0)
- moved C6 0.66 mm to (47.5, 46.5)
- moved C7 0.36 mm to (47.8, 48.2)
- moved L1 0.30 mm to (44.2, 46.5)
- moved C1 0.15 mm to (40.8, 52.5)
Routing:
- net GND: track 79.2 -> 136.8 mm, vias 47 -> 71
- net NRST: track 69.2 -> 80.6 mm, vias 4 -> 3
- net SWCLK: track 46.6 -> 50.1 mm
- net +3V3: track 349.7 -> 353.0 mm, vias 16 -> 17
- net SWDIO: track 48.7 -> 51.8 mm
- net SDA: track 156.1 -> 158.7 mm
- net SCL: track 153.0 -> 155.2 mm
- net SWO: track 46.4 -> 48.3 mm
- net /VBAT: track 23.1 -> 24.2 mm

Commit message: Finishing
Parts:
- moved R8 4.15 mm to (84.0, 58.2), turned to 90 degrees
- moved R9 2.93 mm to (81.4, 58.2), turned to -90 degrees
Routing:
- net +3V3: track 353.0 -> 343.9 mm, vias 17 -> 15
- net SDA: track 158.7 -> 156.0 mm
- net SCL: track 155.2 -> 152.7 mm
- net GND: track 136.8 -> 137.5 mm, vias 71 -> 69

Commit message: fixes
Parts:
- Y1: value 16Hz -> 16MHz
- moved C11 1.72 mm to (43.0, 49.6)
- moved L1 0.74 mm to (44.8, 46.0), turned to -90 degrees
Connections:
- U5 pad 44: WIFI_RESET -> SDIO_POWER_ENABLE
- U5 pad 45: WIFI_ENABLE -> SDIO_DETECT
- U5 pad 56: unconnected-(U5-PB4-Pad56) -> WIFI_ENABLE
- U5 pad 57: unconnected-(U5-PB5-Pad57) -> WIFI_RESET
- U5 pad 61: SDIO_DETECT -> unconnected-(U5-PB8-Pad61)
- U5 pad 62: SDIO_POWER_ENABLE -> unconnected-(U5-PB9-Pad62)
Routing:
- net SDIO_POWER_ENABLE: track 46.2 -> 32.4 mm
- net SDIO_DETECT: track 52.8 -> 40.6 mm
- net WIFI_RESET: track 78.8 -> 70.9 mm
- net WIFI_ENABLE: track 75.5 -> 69.8 mm
- net NRST: track 80.6 -> 78.5 mm
- net GND: track 137.5 -> 139.4 mm, vias 69 -> 70
- net Net-(R10-Pad2): track 74.7 -> 72.9 mm
- net Net-(R11-Pad2): track 64.6 -> 62.9 mm
- net +3V3: track 343.9 -> 342.2 mm
- net Net-(R12-Pad2): track 59.6 -> 58.0 mm
- net +BATT: track 80.1 -> 81.6 mm
- net Net-(R13-Pad2): track 61.7 -> 60.6 mm
- net SCL: track 152.7 -> 153.7 mm
- net SCD30_READY: track 57.9 -> 58.9 mm
- net SDA: track 156.0 -> 156.9 mm
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Other:
- board text added: "HPMA"

Commit message: Finishing touhches on main board
Parts:
- added C23: 100n, Capacitor_SMD:C_0603_1608Metric, F.Cu at (42.0, 32.8)
- added C24: 10n, Capacitor_SMD:C_0805_2012Metric, F.Cu at (43.5, 32.9)
- added C25: 22u, Capacitor_SMD:CP_Elec_6.3x5.8, F.Cu at (50.8, 28.2)
- C11: moved to B.Cu
- C22: footprint Capacitor_SMD:C_0805_2012Metric -> Capacitor_SMD:C_0603_1608Metric
- D2: value CPU_LED -> LED
- D4: value SD_LED -> LED
- J3: footprint Connector_PinHeader_2.54mm:PinHeader_1x04_P2.54mm_Vertical -> Connector_JST:JST_PH_S4B-PH-SM4-TB_1x04-1MP_P2.00mm_Horizontal
- J6: footprint Connector_PinHeader_2.54mm:PinHeader_1x06_P2.54mm_Vertical -> Connector_JST:JST_PH_S6B-PH-SM4-TB_1x06-1MP_P2.00mm_Horizontal
- L1: footprint Inductor_SMD:L_0805_2012Metric -> Inductor_SMD:L_1206_3216Metric
- moved C10 6.75 mm to (73.4, 45.2)
- moved C11 5.28 mm to (47.5, 46.8), turned to -90 degrees
- moved J6 4.17 mm to (64.4, 25.6), turned to 180 degrees
- moved J3 1.66 mm to (39.0, 25.6), turned to 180 degrees
- moved C3 0.75 mm to (58.8, 53.0)
- moved L1 0.58 mm to (44.5, 46.5), turned to 90 degrees
- moved JP3 0.45 mm to (107.5, 102.2), turned to 180 degrees
Connections:
- JP3 pad 1: /BMP280_VCC -> GND
- JP3 pad 3: GND -> /BMP280_VCC
Routing:
- net +3V3: track 342.2 -> 327.9 mm, vias 15 -> 17
- net NRST: track 78.5 -> 64.7 mm
- net GND: track 139.4 -> 149.2 mm, vias 70 -> 77
- net /VBAT: track 24.2 -> 16.6 mm
- net +5V: track 142.6 -> 148.0 mm
- net HPMA_RX: track 30.4 -> 26.9 mm, vias 1 -> 0
- net HPMA_TX: track 30.0 -> 27.1 mm, vias 1 -> 0
- net SWDIO: track 51.8 -> 54.7 mm, vias 1 -> 2
- net SWO: track 48.3 -> 49.7 mm, vias 1 -> 2
- net SWCLK: track 50.1 -> 51.0 mm, vias 1 -> 2
- net +3.3VA: track 6.99 -> 7.72 mm
Other:
- board text added: "5V"
- board text added: "5V Enable"
- board text added: "BMP/BME280"
- board text added: "Batt+"
- board text added: "E-Ink_Waveshare_4.2"
- board text added: "ESP-12S"
- board text added: "Power"
- board text added: "RX"
- board text added: "SCD30"
- board text added: "SCD40"
- board text added: "TX"
- board text added: "Vdd"
- board text added: "Vusb"
