File: KiCad/EnvSensor-Main-v2.1/EnvSensor-Main-v2.1.kicad_pcb (KiCad board)
At the start: 4 copper layers, 102 x 100 mm, 93 parts, among them J1 Conn_01x02, J2 Conn_01x02, J3 HPMA115C0-003, J4 Conn_01x02, J5 Micro_SD_Card_Det, J6 SWD, J7 I2C, J8 POWER_INPUT, Q1 Si3407DV, Q2 IRLML2502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

Commit message: hpma
Other:
- board text added: "Bugs: 1. Recompute areas 2. C1 - wrong footprint 3. Power connector should have silk on top"
- board text removed: "Bugs: 1. Recompute areas 2. C1 - wrong footprint"
Changed lines of the file:
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@@
     (effects (font (size 1.2 1.2) (thickness 0.2) bold) (justify left))
   )
-  (gr_text "Bugs:\n1. Recompute areas\n2. C1 - wrong footprint" (at -35.6 46.2) (layer "F.SilkS")
+  (gr_text "Bugs:\n1. Recompute areas\n2. C1 - wrong footprint\n3. Power connector should have silk on top" (at -35.6 46.2) (layer "F.SilkS")
     (effects (font (size 1.5 1.5) (thickness 0.3) bold) (justify left top))
   )
