File: KiCad/EnvSensor-Power-v2.1/EnvSensor-Power-v2.1.kicad_pcb (KiCad board)
At the start: 4 copper layers, 102 x 100 mm, 139 parts, among them J1 USB_B_Micro, J2 USB_C_Receptacle_USB2.0, J3 BattSense, J4 3V3 Sense, J5 5V Sense, J6 POWER_OUTPUT, Q1 AO6804A, Q3 ZXMP6A16K, SW1 BATT_SWITCH, SW2 Start, U1 LTC3440, U2 AP9101CK6, U3 MCP1825S-3.3, U4 TPS631000, U5 MCP73843-4.2, U6 MCP1826S-5.0, U7 LTC4052, U8 LM2735YMF

Commit message: Fixes
Parts:
- added C33: 4u7, Capacitor_SMD:C_0805_2012Metric, B.Cu at (65.5, 101.7)
- added C39: 4u7, Capacitor_SMD:C_0805_2012Metric, B.Cu at (46.8, 101.8)
- added C40: 4u7, Capacitor_SMD:C_0805_2012Metric, B.Cu at (48.8, 101.8)
- added C5: 4u7, Capacitor_SMD:C_0805_2012Metric, B.Cu at (60.8, 76.9)
- added C7: 4u7, Capacitor_SMD:C_0805_2012Metric, B.Cu at (55.6, 73.3)
- added TS5: TestPoint, TestPoint:TestPoint_THTPad_D1.5mm_Drill0.7mm, B.Cu at (77.2, 83.4)
- added TS8: TestPoint, TestPoint:TestPoint_THTPad_D1.5mm_Drill0.7mm, B.Cu at (79.4, 97.0)
- C10, C8, C9: value 10u -> 4u7
- C2: renamed from C3; value 22u -> 4u7; footprint Capacitor_SMD:C_1206_3216Metric -> Capacitor_SMD:C_0805_2012Metric
- C3: renamed from C4; value 22u -> 4u7; footprint Capacitor_SMD:C_1206_3216Metric -> Capacitor_SMD:C_0805_2012Metric
- C30: renamed from C29; value 10u -> 4u7
- C31: renamed from C30; value 10u -> 4u7
- C32: renamed from C2; value 10u -> 4u7
- C4: renamed from C5; value 22u -> 4u7; footprint Capacitor_SMD:C_1206_3216Metric -> Capacitor_SMD:C_0805_2012Metric
- C41: renamed from C37; value 10u -> 4u7
- C42: renamed from C38; value 10u -> 4u7
- L1: value SLF10145T-220M1R9-H / 22u -> MSS7341-473MLD / 47u; footprint Inductor_SMD:L_TDK_SLF10145 -> Inductor_SMD:L_Coilcraft_XAL8080-XXX
- L5: value MSS5131-473MLC / 47u -> MSS7341-473MLD / 47u; footprint Inductor_SMD:L_Coilcraft_XAL8050-223 -> Inductor_SMD:L_Coilcraft_XAL8080-XXX
- U8: value LM2735YMF -> LM2735XMF
- moved R16 35.0 mm to (86.3, 76.2), turned to 180 degrees
- moved R17 32.9 mm to (86.3, 74.2), turned to 0 degrees
- moved C23 31.0 mm to (81.0, 76.5), turned to 0 degrees
- moved R18 30.9 mm to (86.3, 72.2), turned to 180 degrees
- moved JP6 28.8 mm to (86.3, 70.0), turned to 0 degrees
- moved C22 28.3 mm to (81.0, 74.2), turned to 0 degrees
- moved JP5 26.8 mm to (86.3, 67.5), turned to 180 degrees
- moved U4 25.1 mm to (81.0, 71.5), turned to 90 degrees
- moved L4 22.2 mm to (77.0, 71.4), turned to -90 degrees
- moved C21 21.9 mm to (81.0, 68.5), turned to 0 degrees
- moved C12 20.8 mm to (53.2, 64.7)
- moved C20 19.7 mm to (81.0, 66.2), turned to 0 degrees
- moved C11 17.0 mm to (55.0, 64.7)
- moved D3 14.3 mm to (65.6, 75.8), turned to 90 degrees
- moved TS4 14.1 mm to (69.8, 58.6)
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- renumbered C6 to C15, C15 to C16, C16 to C17, C17 to C18, C18 to C19, C19 to C20, C20 to C21, C21 to C22, C22 to C23, C23 to C24, C24 to C25, C25 to C26, C26 to C27, C27 to C28, C28 to C29, C33 to C34, C31 to C36, C34 to C37, C36 to C38, C40 to C43, C41 to C44, C43 to C45, C42 to C46, C7 to C6, D15 to D10, D5 to D4, D6 to D5, D4 to D6, D13 to D8, D14 to D9, JP8 to JP7, JP9 to JP8, JP7 to JP9, Q3 to Q2, R20 to R18, R22 to R20, R23 to R21, R24 to R22, R25 to R23, R26 to R24, R21 to R25, R29 to R26, R30 to R27, R31 to R28, R32 to R29, R33 to R30, R34 to R31, TS5 to TS6, TS6 to TS7, TS7 to TS9
Routing:
- net /BATT_3V3_FILTER: track 58.5 -> 75.2 mm, vias 0 -> 2
- net /3V7_NOT_REG: track 68.0 -> 78.7 mm, vias 2 -> 0
- net GND: track 144.1 -> 154.7 mm, vias 62 -> 64
- net /3V3_LTC_SW2: track 13.0 -> 17.1 mm
- net /3V3_LTC_SW1: track 13.4 -> 16.2 mm
- net /3V3_FILTER: track 8.96 -> 11.6 mm
- net /5V5_FILTERED: track 9.38 -> 11.8 mm
- net /3V3_LTC_VC: track 3.88 -> 6.19 mm
- net /3V3_LTC_MODE: track 9.74 -> 12.0 mm
- net Net-(C11-Pad1): track 5.02 -> 3.82 mm
- net POWER_5V_ENABLE: track 54.8 -> 53.8 mm
- net /5V_IN: track 12.7 -> 13.6 mm
- net /5V_SW: track 3.42 -> 4.17 mm
- net /3V3_LTC_FB: track 7.10 -> 7.75 mm

Commit message: More fixes
Parts:
- L1, L5: footprint Inductor_SMD:L_Coilcraft_XAL8080-XXX -> Inductor_SMD:L_Coilcraft_XAL7050-XXX
- SW2: moved to B.Cu
- moved SW2 9.53 mm to (33.8, 107.0), turned to 90 degrees
- moved J6 1.69 mm to (111.0, 115.0)
Routing:
- net -BATT: track 74.5 -> 78.0 mm
- net +3V3: track 37.6 -> 38.8 mm
- net +5V: track 22.1 -> 23.1 mm
- net GND: track 154.7 -> 155.2 mm

Commit message: More fixes
Parts:
- D1: footprint Diode_SMD:D_SOD-323 -> Diode_SMD:D_SOD-323_HandSoldering
- L1, L5: footprint Inductor_SMD:L_Coilcraft_XAL7050-XXX -> Inductor_SMD:L_Bourns-SRN8040_8x8.15mm
- L4: footprint Inductor_SMD:L_1210_3225Metric -> Inductor_SMD:L_0805_2012Metric
- moved D1 2.19 mm to (29.8, 51.6)
- moved L5 0.40 mm to (53.6, 94.6)
- moved L1 0.20 mm to (69.4, 69.0)

Commit message: More work
Parts:
- C1, D1, J1, J2: moved to F.Cu
- J3, J4, J5: footprint Connector_PinHeader_2.54mm:PinHeader_1x02_P2.54mm_Vertical -> Connector_PinHeader_2.54mm:PinHeader_1x02_P2.54mm_Horizontal; moved to B.Cu
- R1, R2: moved to B.Cu
- moved SW1 74.5 mm to (27.0, 44.3), turned to -90 degrees
- moved JP1 67.0 mm to (32.8, 24.6), turned to 180 degrees
- moved J3 65.9 mm to (31.5, 22.8), turned to -90 degrees
- moved J1 29.7 mm to (22.4, 75.2), turned to -90 degrees
- moved D1 20.8 mm to (26.6, 72.2), turned to -90 degrees
- moved C1 17.7 mm to (23.6, 69.2)
- moved D5 15.1 mm to (23.1, 86.5)
- moved JP7 15.1 mm to (29.6, 88.8)
- moved JP8 15.1 mm to (29.6, 86.8)
- moved D4 15.1 mm to (25.2, 87.8)
- moved R19 15.1 mm to (27.0, 87.8)
- moved D7 14.6 mm to (23.1, 96.6)
- moved D6 14.6 mm to (25.2, 97.9)
- moved R25 14.6 mm to (27.0, 97.9)
- moved C43 10.0 mm to (42.2, 79.2)
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Connections:
- J3 pad 2: +BATT -> /BATT_BARE
- J4 pad 1: /3V3_REG -> +3V3
- J4 pad 2: +3V3 -> /3V3_REG
- J5 pad 1: /5V_REG -> +5V
- J5 pad 2: +5V -> /5V_REG
- JP1 pad 1: /BATT_SW -> /BATT_BARE
- JP1 pad 2: +BATT -> /BATT_SW
- SW1 pad 1: unconnected-(SW1-A-Pad1) -> /BATT_SW
- SW1 pad 2: /BATT_SW -> +BATT
- SW1 pad 3: /BATT_BARE -> unconnected-(SW1-C-Pad3)
Routing:
- net -BATT: track 78.0 -> 58.5 mm
- net /BATT_SW: track 6.64 -> 23.4 mm
- net VBUS: track 252.9 -> 265.9 mm
- net +BATT: track 217.3 -> 204.9 mm
- net /CHRG_ACPR: track 55.5 -> 66.1 mm
- net /CHRG_CHRG: track 100.4 -> 110.7 mm
- net /5V_IN: track 14.0 -> 20.6 mm
- net /BATT_3V3_FILTER: track 75.2 -> 71.5 mm
- net /BATT_BARE: track 59.9 -> 63.0 mm
- net +5V: track 23.1 -> 25.4 mm
- net +3V3: track 38.8 -> 40.2 mm
- net /BATT2-: track 8.23 -> 7.03 mm
- net /3V7_NOT_REG: track 78.7 -> 79.8 mm
- net /BATT3-: track 8.23 -> 7.14 mm
- net /5V_REG: track 16.0 -> 17.0 mm
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- added copper zone on F.Cu, net /USB_SHIELD
- removed copper zone on B.Cu, net /USB_SHIELD
