File: KiCad/EnvSensor-Power-v2.1/EnvSensor-Power-v2.1.kicad_sch (KiCad schematic)
At the start: 146 parts, among them J1 USB_B_Micro, J2 USB_C_Receptacle_USB2.0, J3 BattSense, J4 3V3 Sense, J5 5V Sense, J6 POWER_OUTPUT, Q1 AO6804A, Q2 ZXMP6A16K, SW1 BATT_SWITCH, SW2 Start, U1 LTC3440, U2 AP9101CK6, U3 MCP1825S-3.3, U4 TPS631000, U5 MCP73843-4.2, U6 MCP1826S-5.0, U7 LTC4052, U8 LM2735XMF

Commit message: More work
Parts:
- J3, J4, J5: footprint Connector_PinHeader_2.54mm:PinHeader_1x02_P2.54mm_Vertical -> Connector_PinHeader_2.54mm:PinHeader_1x02_P2.54mm_Horizontal
Connections:
- net +3V3: now also J4.1 (Pin_1); no longer J4.2 (Pin_2)
- net +5V: now also J5.1 (Pin_1); no longer J5.2 (Pin_2)
- net +BATT: now also SW1.2 (B); no longer J3.2 (Pin_2), JP1.2
- net 3V3_REG: now also J4.2 (Pin_2); no longer J4.1 (Pin_1)
- net 5V_REG: now also J5.2 (Pin_2); no longer J5.1 (Pin_1)
- net BATT_BARE: now also J3.2 (Pin_2), JP1.1; no longer SW1.3 (C)
- net BATT_SW: now also JP1.2, SW1.1 (A); no longer JP1.1, SW1.2 (B)
- no-connect marks 11 -> 10
Other:
- moved on the sheet: J3, J4, J5, JP1, SW1
Changed lines of the file:
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@@
   (junction (at 354.33 142.24) (diameter 0) (color 0 0 0 0)
   )
-  (junction (at 321.945 142.24) (diameter 0) (color 0 0 0 0)
+  (junction (at 41.91 129.54) (diameter 0) (color 0 0 0 0)
   )
-  (junction (at 61.595 127) (diameter 0) (color 0 0 0 0)
+  (junction (at 321.945 142.24) (diameter 0) (color 0 0 0 0)
   )
   (junction (at 378.46 135.89) (diameter 0) (color 0 0 0 0)
   )
-  (junction (at 69.215 127) (diameter 0) (color 0 0 0 0)
-  )
   (junction (at 365.76 293.37) (diameter 0) (color 0 0 0 0)
   )
@@
   (junction (at 355.6 135.89) (diameter 0) (color 0 0 0 0)
   )
+  (junction (at 49.53 129.54) (diameter 0) (color 0 0 0 0)
+  )
   (junction (at 139.7 161.29) (diameter 0) (color 0 0 0 0)
   )
@@
   )
   (no_connect (at 114.3 48.26))
-  (no_connect (at 53.34 121.92))
+  (no_connect (at 58.42 129.54))
   (no_connect (at 57.15 46.99))
-  (no_connect (at 43.18 124.46))
   (no_connect (at 114.3 50.8))
   (no_connect (at 57.15 49.53))
@@
     (stroke (width 0) (type default))
   )
+  (wire (pts (xy 50.8 129.54) (xy 50.8 124.46))
+    (stroke (width 0) (type default))
+  )
   (wire (pts (xy 467.995 179.07) (xy 467.995 181.61))
     (stroke (width 0) (type default))
@@
     (stroke (width 0) (type default))
   )
-  (wire (pts (xy 64.135 125.73) (xy 64.135 127))
+  (wire (pts (xy 44.45 125.73) (xy 44.45 127))
     (stroke (width 0) (type default))
   )
@@
     (stroke (width 0) (type default))
   )
+  (wire (pts (xy 68.58 127) (xy 72.39 127))
+    (stroke (width 0) (type default))
+  )
   (wire (pts (xy 369.57 129.54) (xy 378.46 129.54))
     (stroke (width 0) (type default))
@@
     (stroke (width 0) (type default))
   )
-  (wire (pts (xy 67.945 129.54) (xy 69.215 129.54))
+  (wire (pts (xy 48.26 129.54) (xy 49.53 129.54))
     (stroke (width 0) (type default))
   )
@@
     (stroke (width 0) (type default))
   )
-  (wire (pts (xy 66.675 127) (xy 69.215 127))
+  (wire (pts (xy 46.99 127) (xy 49.53 127))
     (stroke (width 0) (type default))
   )
@@
     (stroke (width 0) (type default))
   )
-  (wire (pts (xy 69.215 129.54) (xy 69.215 127))
+  (wire (pts (xy 49.53 129.54) (xy 49.53 127))
     (stroke (width 0) (type default))
   )
@@
     (stroke (width 0) (type default))
   )
-  (wire (pts (xy 61.595 127) (xy 64.135 127))
+  (wire (pts (xy 41.91 127) (xy 44.45 127))
     (stroke (width 0) (type default))
   )
@@
     (stroke (width 0) (type default))
   )
-  (wire (pts (xy 61.595 127) (xy 61.595 129.54))
+  (wire (pts (xy 41.91 127) (xy 41.91 129.54))
     (stroke (width 0) (type default))
   )
@@
     (stroke (width 0) (type default))
   )
+  (wire (pts (xy 50.8 124.46) (xy 58.42 124.46))
+    (stroke (width 0) (type default))
+  )
   (wire (pts (xy 113.03 279.4) (xy 118.11 279.4))
     (stroke (width 0) (type default))
@@
     (stroke (width 0) (type default))
   )
-  (wire (pts (xy 66.675 125.73) (xy 66.675 127))
+  (wire (pts (xy 46.99 125.73) (xy 46.99 127))
     (stroke (width 0) (type default))
   )
@@
     (stroke (width 0) (type default))
   )
-  (wire (pts (xy 41.91 129.54) (xy 43.18 129.54))
-    (stroke (width 0) (type default))
-  )
   (wire (pts (xy 388.62 135.89) (xy 400.05 135.89))
     (stroke (width 0) (type default))
@@
     (stroke (width 0) (type default))
   )
+  (wire (pts (xy 49.53 129.54) (xy 50.8 129.54))
+    (stroke (width 0) (type default))
+  )
   (wire (pts (xy 307.975 142.24) (xy 316.23 142.24))
     (stroke (width 0) (type default))
@@
     (stroke (width 0) (type default))
   )
-  (wire (pts (xy 62.865 129.54) (xy 61.595 129.54))
+  (wire (pts (xy 43.18 129.54) (xy 41.91 129.54))
     (stroke (width 0) (type default))
   )
@@
     (stroke (width 0) (type default))
   )
-  (wire (pts (xy 53.34 127) (xy 61.595 127))
-    (stroke (width 0) (type default))
-  )
   (wire (pts (xy 267.97 193.04) (xy 267.97 196.85))
     (stroke (width 0) (type default))
@@
     (stroke (width 0) (type default))
   )
-  (wire (pts (xy 69.215 127) (xy 72.39 127))
-    (stroke (width 0) (type default))
-  )
   (wire (pts (xy 502.92 309.88) (xy 511.81 309.88))
     (stroke (width 0) (type default))
@@
     (effects (font (size 1.27 1.27)) (justify left bottom))
   )
-  (label "BATT_SW" (at 54.61 127 0) (fields_autoplaced)
+  (label "BATT_SW" (at 50.8 124.46 0) (fields_autoplaced)
     (effects (font (size 1.27 1.27)) (justify left bottom))
   )
@@
     )
   )
-  (symbol (lib_id "Connector_Generic:Conn_01x02") (at 527.05 173.99 90) (unit 1)
+  (symbol (lib_id "Connector_Generic:Conn_01x02") (at 529.59 173.99 270) (mirror x) (unit 1)
     (in_bom yes) (on_board yes) (dnp no)
-    (property "Reference" "J4" (at 527.2532 171.958 0)
+    (property "Reference" "J4" (at 529.3868 171.958 0)
       (effects (font (size 1.27 1.27)) (justify left))
     )
-    (property "Value" "3V3 Sense" (at 529.5646 171.958 0)
+    (property "Value" "3V3 Sense" (at 527.0754 171.958 0)
       (effects (font (size 1.27 1.27)) (justify left))
     )
-    (property "Footprint" "Connector_PinHeader_2.54mm:PinHeader_1x02_P2.54mm_Vertical" (at 527.05 173.99 0)
+    (property "Footprint" "Connector_PinHeader_2.54mm:PinHeader_1x02_P2.54mm_Horizontal" (at 529.59 173.99 0)
       (effects (font (size 1.27 1.27)) hide)
     )
-    (property "Datasheet" "~" (at 527.05 173.99 0)
+    (property "Datasheet" "~" (at 529.59 173.99 0)
       (effects (font (size 1.27 1.27)) hide)
     )
@@
     )
   )
-  (symbol (lib_id "Connector_Generic:Conn_01x02") (at 440.69 276.86 90) (unit 1)
+  (symbol (lib_id "Connector_Generic:Conn_01x02") (at 443.23 276.86 270) (mirror x) (unit 1)
     (in_bom yes) (on_board yes) (dnp no)
-    (property "Reference" "J5" (at 440.8932 274.828 0)
+    (property "Reference" "J5" (at 443.0268 274.828 0)
       (effects (font (size 1.27 1.27)) (justify left))
     )
-    (property "Value" "5V Sense" (at 443.2046 274.828 0)
+    (property "Value" "5V Sense" (at 440.7154 274.828 0)
       (effects (font (size 1.27 1.27)) (justify left))
     )
-    (property "Footprint" "Connector_PinHeader_2.54mm:PinHeader_1x02_P2.54mm_Vertical" (at 440.69 276.86 0)
+    (property "Footprint" "Connector_PinHeader_2.54mm:PinHeader_1x02_P2.54mm_Horizontal" (at 443.23 276.86 0)
       (effects (font (size 1.27 1.27)) hide)
     )
-    (property "Datasheet" "~" (at 440.69 276.86 0)
+    (property "Datasheet" "~" (at 443.23 276.86 0)
       (effects (font (size 1.27 1.27)) hide)
     )
@@
     )
   )
-  (symbol (lib_id "Connector_Generic:Conn_01x02") (at 64.135 120.65 90) (unit 1)
+  (symbol (lib_id "Connector_Generic:Conn_01x02") (at 46.99 120.65 270) (mirror x) (unit 1)
     (in_bom yes) (on_board yes) (dnp no)
-    (property "Reference" "J3" (at 69.215 119.38 90)
+    (property "Reference" "J3" (at 41.91 119.38 90)
       (effects (font (size 1.27 1.27)) (justify right))
     )
-    (property "Value" "BattSense" (at 69.215 121.92 90)
+    (property "Value" "BattSense" (at 41.91 121.92 90)
       (effects (font (size 1.27 1.27)) (justify right))
     )
-    (property "Footprint" "Connector_PinHeader_2.54mm:PinHeader_1x02_P2.54mm_Vertical" (at 64.135 120.65 0)
+    (property "Footprint" "Connector_PinHeader_2.54mm:PinHeader_1x02_P2.54mm_Horizontal" (at 46.99 120.65 0)
       (effects (font (size 1.27 1.27)) hide)
     )
-    (property "Datasheet" "~" (at 64.135 120.65 0)
+    (property "Datasheet" "~" (at 46.99 120.65 0)
       (effects (font (size 1.27 1.27)) hide)
     )
@@
     )
   )
-  (symbol (lib_id "EnvSensor-v2-rescue:Jumper_NO_Small-Device") (at 65.405 129.54 0) (unit 1)
+  (symbol (lib_id "EnvSensor-v2-rescue:Jumper_NO_Small-Device") (at 45.72 129.54 0) (unit 1)
     (in_bom yes) (on_board yes) (dnp no)
-    (property "Reference" "JP1" (at 69.215 132.08 0)
+    (property "Reference" "JP1" (at 49.53 132.08 0)
       (effects (font (size 1.27 1.27)))
     )
-    (property "Value" "NO" (at 65.405 132.08 0)
+    (property "Value" "NO" (at 45.72 132.08 0)
       (effects (font (size 1.27 1.27)))
     )
-    (property "Footprint" "Jumper:SolderJumper-2_P1.3mm_Open_RoundedPad1.0x1.5mm" (at 65.405 129.54 0)
+    (property "Footprint" "Jumper:SolderJumper-2_P1.3mm_Open_RoundedPad1.0x1.5mm" (at 45.72 129.54 0)
       (effects (font (size 1.27 1.27)) hide)
     )
-    (property "Datasheet" "~" (at 65.405 129.54 0)
+    (property "Datasheet" "~" (at 45.72 129.54 0)
       (effects (font (size 1.27 1.27)) hide)
     )
@@
     )
   )
-  (symbol (lib_id "Switch:SW_SPDT") (at 48.26 127 0) (mirror y) (unit 1)
+  (symbol (lib_id "Switch:SW_SPDT") (at 63.5 127 0) (mirror y) (unit 1)
     (in_bom yes) (on_board yes) (dnp no)
-    (property "Reference" "SW1" (at 49.53 129.54 0)
+    (property "Reference" "SW1" (at 64.77 129.54 0)
       (effects (font (size 1.27 1.27)))
     )
-    (property "Value" "BATT_SWITCH" (at 46.99 121.92 0)
+    (property "Value" "BATT_SWITCH" (at 66.04 121.92 0)
       (effects (font (size 1.27 1.27)))
     )
-    (property "Footprint" "Button_Switch_THT:SW_Lever_1P2T_NKK_GW12LxH" (at 48.26 127 0)
+    (property "Footprint" "Button_Switch_THT:SW_Lever_1P2T_NKK_GW12LxH" (at 63.5 127 0)
       (effects (font (size 1.27 1.27)) hide)
     )
-    (property "Datasheet" "~" (at 48.26 127 0)
+    (property "Datasheet" "~" (at 63.5 127 0)
       (effects (font (size 1.27 1.27)) hide)
     )

Commit message: Finish
Parts:
- added C47, C48, C49, C50: Cx, Capacitor_SMD:C_0805_2012Metric, symbol Device:C
- added R32, R33, R34, R35: Rx, Resistor_SMD:R_0805_2012Metric, symbol Device:R
- added TS10, TS11, TS12, TS13, TS14, TS15: TestPoint, TestPoint:TestPoint_THTPad_D1.5mm_Drill0.7mm, symbol Connector:TestPoint
Connections:
- net 3V3_FILTER: now also C47.1
- net 3V3_REG: now also TS13.1
- net 5V5_FILTERED: now also C48.1
- net 5V_IN: now also C50.1
- net 5V_REG: now also TS11.1
- net BATT_3V3_FILTER: now also C49.1
- net GND: now also R32.1, R33.1, R34.1, R35.1, TS10.1, TS12.1, TS14.1, TS15.1
- new net: C50.2, R35.2
- new net: C47.2, R32.2
- new net: C48.2, R33.2
- new net: C49.2, R34.2
Other:
- moved on the sheet: C13, C17, C29, C30, C31, C32, C33, C34, C35, C36, C37, C39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
