File: KiCad/EnvSensor-Power-v2.1/EnvSensor-Power-v2.1.kicad_sch (KiCad schematic)
At the start: 160 parts, among them J1 USB_B_Micro, J2 USB_C_Receptacle_USB2.0, J3 BattSense, J4 3V3 Sense, J5 5V Sense, J6 POWER_OUTPUT, Q1 AO6804A, Q2 ZXMP6A16K, SW1 BATT_SWITCH, SW2 Start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

Commit message: c++ project for 2.1 introduced
Parts:
- R19, R25, R27: value 3k3 -> 5k
Other:
- note added: "1. Each part should allow to measure its power consumption 2. Enhancements from v1. 1. Reset button 2. Button to start battery protection after power loss 3. Solution to measure voltage at battery Bugs 1. Too big caps around LDOs"
- note added: "I=15mA Vpp=170mV I=110mA Vpp=40mV"
- note added: "I=5V/5kR=1mA"
- note added: "Measurements f=1.6MHz"
- note removed: "1. Each part should allow to measure its power consumption 2. Enhancements from v1. 1. Reset button 2. Button to start battery protection after power loss 3. Solution to measure voltage at battery"
Changed lines of the file:
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@@
     (effects (font (size 1.27 1.27)) (justify left bottom))
   )
-  (text "1. Each part should allow to measure its power consumption\n2.\n\nEnhancements from v1.\n1. Reset button\n2. Button to start battery protection after power loss\n3. Solution to measure voltage at battery"
+  (text "1. Each part should allow to measure its power consumption\n2.\n\nEnhancements from v1.\n1. Reset button\n2. Button to start battery protection after power loss\n3. Solution to measure voltage at battery\n\nBugs\n1. Too big caps around LDOs"
     (at -102.87 7.62 0)
     (effects (font (size 1.27 1.27)) (justify left bottom))
@@
     (effects (font (size 1.27 1.27)) (justify left bottom))
   )
+  (text "I=15mA    Vpp=170mV\nI=110mA    Vpp=40mV" (at 410.21 120.65 0)
+    (effects (font (size 1.27 1.27)) (justify left bottom))
+  )
   (text "Li-Ion 1 cell 4.2V" (at 106.68 308.61 0)
     (effects (font (size 1.27 1.27)) (justify left bottom))
@@
     (effects (font (size 1.1176 1.1176)) (justify left bottom))
   )
+  (text "I=5V/5kR=1mA" (at 501.65 287.02 0)
+    (effects (font (size 1.27 1.27)) (justify left bottom))
+  )
   (text "Cout=1*47u" (at 394.97 207.01 0)
     (effects (font (size 1.27 1.27)) (justify left bottom))
@@
     (effects (font (size 1.27 1.27)) (justify left bottom))
   )
+  (text "Measurements\nf=1.6MHz" (at 254 260.35 0)
+    (effects (font (size 1.27 1.27)) (justify left bottom))
+  )
   (label "3V3_LTC_MODE" (at 342.9 148.59 0) (fields_autoplaced)
     (effects (font (size 1.27 1.27)) (justify left bottom))
@@
       (effects (font (size 1.27 1.27)) (justify right))
     )
-    (property "Value" "3k3" (at 206.248 241.173 0)
+    (property "Value" "5k" (at 206.248 241.173 0)
       (effects (font (size 1.27 1.27)) (justify right))
     )
@@
       (effects (font (size 1.27 1.27)) (justify right))
     )
-    (property "Value" "3k3" (at 206.248 289.433 0)
+    (property "Value" "5k" (at 206.248 289.433 0)
       (effects (font (size 1.27 1.27)) (justify right))
     )
@@
       (effects (font (size 1.27 1.27)) (justify right))
     )
-    (property "Value" "3k3" (at 495.808 288.163 0)
+    (property "Value" "5k" (at 495.808 288.163 0)
       (effects (font (size 1.27 1.27)) (justify right))
     )
